File: hardware/interface-board/MEP-MAXI-85V-1-REV-2-Interface-Board.kicad_pcb (KiCad board)
At the start: 4 copper layers, 160 x 128.5 mm, 204 parts, among them IC401 AT24C256C-MAHL-E, IC701 LTV-846S, IC702 LTV-846S, IC703 LTV-846S, IC704 LTV-846S, IC801 LTV-846S, J201 Conn_02x07_Odd_Even, J301 Barrel_Jack_MountingPin, J408 Conn_01x04, J501 Screw_Terminal_01x02, J601 Conn_02x10_Odd_Even, Q501 IRFR7540TRPBF, Q502 IRFR7540TRPBF, Q503 IRFR7540TRPBF, Q504 IRFR7540TRPBF, Q505 IRFR7540TRPBF, Q506 IRFR7540TRPBF, Q507 IRFR7540TRPBF, Q508 IRFR7540TRPBF, Q509 IRFR7540TRPBF, Q510 IRFR7540TRPBF, Q701 BSS138 JI, Q702 BSS138 JI, Q703 BSS138 JI, Q704 BSS138 JI, Q705 BSS138 JI, Q706 BSS138 JI, Q707 BSS138 JI, Q708 BSS138 JI, Q709 BSS138 JI, Q710 BSS138 JI, Q711 BSS138 JI, Q712 BSS138 JI, Q713 BSS138 JI, Q714 BSS138 JI, Q715 BSS138 JI, Q716 BSS138 JI, Q801 BSS138 JI, U301 LM1084-ADJ, U302 LM1084-ADJ, U303 LM1084-ADJ

Commit message: X1 Release
Released X1 revision for both the interface board and the input test fixture breakout board.
Parts:
- J501: footprint TerminalBlock:TerminalBlock_Altech_AK300-2_P5.00mm -> TerminalBlock:TerminalBlock_bornier-2_P5.08mm
- moved J501 2.94 mm to (155.3, 36.2)
- moved J601 0.48 mm to (195.8, 36.5)
- moved Q716 0.18 mm to (121.9, 115.7)
Routing:
- net +3V3: track 547.2 -> 680.0 mm, vias 54 -> 56
- net /Solenoid MOSFETS/FUSED_GND: track 17.2 -> 39.1 mm
- net 24VRAW: track 231.5 -> 240.1 mm
- net /Photoisolators/ESTOP: track 178.5 -> 186.6 mm
- net /Arduino DUE IO/D44: track 147.3 -> 141.3 mm
- net /Output Connections/SOL_FEED_REVERSE: track 49.0 -> 45.5 mm
- net /Photoisolators/AUTO_BUTTON: track 113.6 -> 117.0 mm
- net /Arduino DUE IO/D36: track 167.8 -> 165.1 mm
- net GND: track 0.00 -> 1.50 mm, vias 42 -> 65
- net /Arduino DUE IO/D40: track 181.1 -> 179.8 mm
- net /Photoisolators/PROXIMITY_SHEAR_HOME: track 122.6 -> 123.8 mm
- net /Photoisolators/SHEAR_BUTTON: track 142.6 -> 143.7 mm
- net /Arduino DUE IO/D37: track 174.9 -> 173.9 mm
- net /Arduino DUE IO/D45: track 158.1 -> 157.2 mm
- net /Arduino DUE IO/D47: track 179.6 -> 178.6 mm
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- added copper zone on B.Cu, net +3V3
- added copper zone on In1.Cu, net +3V3
- added copper zone on In2.Cu, net +3V3
- added copper zone on B.Cu, net +5V
- added copper zone on In2.Cu, net +5V
Other:
- board text added: "/JGilcreast/MetalHead"
- board text added: "Interface Board Hardware: Connor McMillan Firmware: John Gilcreast Rev X1"
- board text added: "METALHEAD"
- board text removed: "/username/open85V"
- board text removed: "Hardware: Connor McMillan Firmware: John Gilcreast"
- board text removed: "OPEN 85V"
- board text removed: "REV X1"
