File: hardware/interface-board/MEP-MAXI-85V-1-REV-2-Interface-Board.kicad_pcb (KiCad board)
At the start: 4 copper layers, 221.5 x 130.8 mm, 407 parts, among them IC401 AT24C256C-MAHL-E, IC701 LTV-846S, IC702 LTV-846S, IC703 LTV-846S, IC704 LTV-846S, IC705 LTV-846S, J201 USB_C_Receptacle_USB2.0_16P, J202 Conn_02x07_Odd_Even, J203 Screw_Terminal_01x02, J301 Barrel_Jack_MountingPin, J401 TC2030, J501 Conn_02x10_Odd_Even, J502 Screw_Terminal_01x02, J601 USB_C_Receptacle_USB2.0_16P, J602 RJ45_Amphenol_RJMG1BD3B8K1ANR, J603 Conn_02x05_Odd_Even, J604 Conn_Coaxial, J605 Conn_01x24_MountingPin, Q201 IRFR7540TRPBF, Q202 IRFR7540TRPBF, Q203 IRFR7540TRPBF, Q204 IRFR7540TRPBF, Q205 IRFR7540TRPBF, Q206 IRFR7540TRPBF, Q207 IRFR7540TRPBF, Q208 IRFR7540TRPBF, Q209 IRFR7540TRPBF, Q210 IRFR7540TRPBF, Q401 DMP3099L, Q601 BSS138 JI, Q701 BSS138 JI, Q702 BSS138 JI, Q703 BSS138 JI, Q704 BSS138 JI, Q705 BSS138 JI, Q706 BSS138 JI, Q707 BSS138 JI, Q708 BSS138 JI, Q709 BSS138 JI, Q710 BSS138 JI, Q711 BSS138 JI, Q712 BSS138 JI, Q713 BSS138 JI, Q714 BSS138 JI, Q715 BSS138 JI, Q716 BSS138 JI, Q717 BSS138 JI, SW401 SW_SPST_Omron_B3FS-100xP, SW601 SW_SPST_Omron_B3FS-100xP, U201 USBLC6-2SC6, U301 LM1084-ADJ, U302 LM1084-ADJ, U303 LM1084-ADJ, U401 ATmega16U2-M, U402 SN74LVC1G125DCK, U403 SN74LVC1G125DCK, U404 ATSAM3X8EA-AU, U601 USBLC6-2SC6, U602 CH340E, U603 RASPBERRY_PI_ZERO_2_W, U701 SN74HC14PWR, U702 SN74HC14PWR, U703 SN74HC14PWR, Y401 16MHz, Y402 12MHz, Y403 32.768MHz

Commit message: [feat] Revert to Arduino + add PHY
Removed Arduino Due integration. Added W5500 ENET PHY
Parts:
- removed the C302 at (68.7, 121.0)
- removed C404, C406, C407, C414, C415, C416, C417, C418, C419, C420, C421, C422, C423, C424, C425, C426, C427, C428, C430, C433, C434, C438, C606: 100nF, Capacitor_SMD:C_0805_2012Metric
- removed C405: 1uF, Capacitor_SMD:C_0805_2012Metric
- removed C408, C409, C411, C412: 22pF, Capacitor_SMD:C_0805_2012Metric
- removed C410: 10pF, Capacitor_SMD:C_0805_2012Metric
- removed C413: 10nF, Capacitor_SMD:C_0805_2012Metric
- removed C429, C431, C432, C435, C436, C437: 4.7uF, Capacitor_SMD:C_0805_2012Metric
- removed the C604 at (225.0, 95.1)
- removed the C605 at (222.5, 95.2)
- removed C608, C609: 470uF, Capacitor_SMD:CP_Elec_4x5.4
- removed the C717 at (149.9, 101.7)
- removed C720, C721, C722: 47uF, Capacitor_SMD:C_0805_2012Metric
- removed the D301 at (37.5, 130.0)
- removed the D302 at (37.6, 136.8)
- removed the D304 at (58.0, 139.5)
- removed D305: SS10100, Diode_SMD:D_SMC
- removed D307: WHITE, LED_SMD:LED_1210_3225Metric
- removed D309: GREEN, LED_SMD:LED_1210_3225Metric
- removed D311: YELLOW, LED_SMD:LED_1210_3225Metric
- removed D401: 1N4148W, Diode_SMD:D_SOD-323
- removed D402: YELLOW, LED_SMD:LED_1206_3216Metric
- removed D403, D601: GREEN, LED_SMD:LED_1206_3216Metric
- removed D602: SS34, Diode_SMD:D_SMA
- removed D701, D702, D703, D704, D705, D706, D707, D708, D709, D710, D711, D712, D713, D714, D715, D716: BLUE, LED_SMD:LED_1210_3225Metric
- removed D717: RED, LED_SMD:LED_1210_3225Metric
- removed F501: 3512P, Fuse:Fuseholder_Clip-5x20mm_Keystone_3512P_Inline_P23.62x7.27mm_D1.02x2.41x1.02x1.57mm_Horizontal
- removed the J201 at (78.5, 144.9)
- removed J203, J502: Screw_Terminal_01x02, TerminalBlock:TerminalBlock_bornier-2_P5.08mm
- removed J401: TC2030, Connector:Tag-Connect_TC2030-IDC-NL_2x03_P1.27mm_Vertical
- removed the J601 at (231.9, 66.7)
- removed the J602 at (219.0, 47.3)
- removed JP201, JP202: Jumper_3_Open, Connector_PinHeader_2.54mm:PinHeader_1x03_P2.54mm_Vertical
- removed L201, L301, L601: 470uH, Inductor_SMD:L_12x12mm_H8mm
- removed L401, L402, L403: 10uH, Inductor_SMD:L_0805_2012Metric
- removed Q701, Q702, Q703, Q704, Q705, Q706, Q707, Q708, Q709, Q710, Q711, Q712, Q713, Q714, Q715, Q716, Q717: BSS138 JI, Package_TO_SOT_SMD:SOT-23
- removed the R222 at (85.0, 139.0)
- removed the R307 at (25.8, 108.3)
- removed the R311 at (53.2, 94.9)
- removed the R401 at (81.7, 88.2)
- removed the R402 at (79.7, 77.2)
- removed the R405 at (63.7, 80.0)
- removed the R406 at (63.7, 78.0)
- removed R409: 6K8, Resistor_SMD:R_0805_2012Metric
- removed R410: 0R, Resistor_SMD:R_0805_2012Metric
- removed R411: 100K, Resistor_SMD:R_0805_2012Metric
- removed R412, R413, R414, R415, R416, R417, R418, R419, R420, R421, R422, R423, R424, R425, R426, R427, R428, R429, R430, R431, R432, R433, R434, R435, R436, R437, R438, R439: 33R, Resistor_SMD:R_0805_2012Metric
- removed R440: 10K, Resistor_SMD:R_0805_2012Metric
- removed R441, R442, R443: 1R, Resistor_SMD:R_0805_2012Metric
- removed the R601 at (220.8, 127.5)
- removed the R602 at (224.5, 98.7)
- removed the R603 at (228.7, 73.2)
- removed the R604 at (228.8, 60.0)
- removed the R705 at (111.9, 39.0)
- removed the R706 at (111.9, 44.0)
- removed the R707 at (111.9, 49.0)
- removed the R708 at (111.9, 54.5)
- removed the R710 at (137.9, 44.0)
- removed the R711 at (137.9, 49.0)
- removed the R715 at (163.9, 48.8)
- removed the R716 at (164.0, 53.8)
- removed the R717 at (189.5, 38.8)
- removed the R718 at (123.1, 63.4)
- removed the R721 at (123.2, 73.4)
- removed the R722 at (123.1, 78.4)
- removed R740, R741, R744, R745, R746, R747, R748, R749, R750, R751: 200R, Resistor_SMD:R_1206_3216Metric
- removed SW401: SW_SPST_Omron_B3FS-100xP, Button_Switch_SMD:SW_SPST_EVQPE1
- removed TP701, TP702, TP703, TP704, TP705, TP717, TP718, TP719, TP720, TP730, TP731, TP732, TP733, TP743, TP744, TP745, TP746: Orange, TestPoint:TestPoint_THTPad_D1.0mm_Drill0.5mm
- removed TP706, TP707, TP708, TP709, TP710, TP721, TP722, TP723, TP724, TP734, TP735, TP736, TP737, TP747, TP748, TP749, TP750: Yellow, TestPoint:TestPoint_THTPad_D1.0mm_Drill0.5mm
- removed TP711, TP712, TP713, TP714, TP715, TP725, TP726, TP727, TP728, TP738, TP739, TP740, TP741, TP751, TP752, TP753, TP754: White, TestPoint:TestPoint_THTPad_D1.0mm_Drill0.5mm
- removed TP716, TP729: Red, TestPoint:TestPoint_THTPad_D3.0mm_Drill1.5mm
- removed TP742, TP755: Black, TestPoint:TestPoint_THTPad_D3.0mm_Drill1.5mm
- removed the U401 at (75.8, 83.5)
- removed the U602 at (218.0, 97.7)
- removed Y401: 16MHz, Crystal:Crystal_SMD_3225-4Pin_3.2x2.5mm
- removed Y402: 12MHz, Crystal:Crystal_SMD_3225-4Pin_3.2x2.5mm
- removed Y403: 32.768MHz, Crystal:Crystal_SMD_3225-4Pin_3.2x2.5mm
- added A401: Arduino_Due_Shield, arduino-library:Arduino_Due_Shield, F.Cu at (86.5, 122.7)
- added C201: 0.1uF, Capacitor_SMD:C_0805_2012Metric, F.Cu at (77.3, 85.7)
- added C304: 330uF 25V, Capacitor_SMD:CP_Elec_8x10.5, F.Cu at (36.3, 93.1)
- added C305: 330uF 25V, Capacitor_SMD:CP_Elec_8x10.5, F.Cu at (23.9, 94.5)
- added C306: 100nF, Capacitor_SMD:C_1206_3216Metric, B.Cu at (23.9, 99.7)
- added C307: 0.1uF, Capacitor_SMD:C_0805_2012Metric, F.Cu at (93.8, 102.6)
- added C310: 330uF 25V, Capacitor_SMD:CP_Elec_8x10.5, F.Cu at (35.4, 112.0)
- added C311: 330uF 25V, Capacitor_SMD:CP_Elec_8x10.5, F.Cu at (23.8, 111.8)
- added C312: 100nF, Capacitor_SMD:C_1206_3216Metric, B.Cu at (23.8, 108.0)
- added C315: 0.1uF, Capacitor_SMD:C_0805_2012Metric, F.Cu at (57.2, 141.9)
- added C316: 100nF, Capacitor_SMD:C_1206_3216Metric, F.Cu at (84.6, 124.6)
- added C603: 100nF, Capacitor_SMD:C_0805_2012Metric, B.Cu at (218.8, 132.0)
- added C716: 1uF, Capacitor_SMD:C_0805_2012Metric, F.Cu at (209.2, 46.6)
- added C901: 10uF, Capacitor_SMD:CP_Elec_4x5.4, F.Cu at (134.5, 107.9)
- added C902: 0.1uF, Capacitor_SMD:C_0805_2012Metric, F.Cu at (131.1, 106.3)
- added C903: 0.1uF, Capacitor_SMD:C_0805_2012Metric, F.Cu at (116.1, 94.3)
- added C904: 0.1uF, Capacitor_SMD:C_0805_2012Metric, B.Cu at (116.1, 94.3)
- added C905: 0.1uF, Capacitor_SMD:C_0805_2012Metric, F.Cu at (112.1, 94.3)
- added C906: 0.1uF, Capacitor_SMD:C_0805_2012Metric, B.Cu at (112.1, 94.3)
- added C907: 0.1uF, Capacitor_SMD:C_0805_2012Metric, F.Cu at (114.1, 94.3)
- added C908: 0.1uF, Capacitor_SMD:C_0805_2012Metric, B.Cu at (114.1, 94.3)
- added C909: 10uF, Capacitor_SMD:CP_Elec_4x5.4, F.Cu at (108.7, 92.5)
- added C910: 6.8nF, Capacitor_SMD:C_0805_2012Metric, F.Cu at (142.6, 129.2)
- added C911: 6.8nF, Capacitor_SMD:C_0805_2012Metric, F.Cu at (140.6, 129.2)
- added C912: 22nF, Capacitor_SMD:C_0805_2012Metric, B.Cu at (109.3, 97.0)
- added C913: 10nF, Capacitor_SMD:C_0805_2012Metric, F.Cu at (107.5, 108.7)
- added C914: 18pF, Capacitor_SMD:C_0805_2012Metric, B.Cu at (135.0, 102.4)
- added C915: 18pF, Capacitor_SMD:C_0805_2012Metric, B.Cu at (132.4, 99.1)
- added C916: 10nF, Capacitor_SMD:C_0805_2012Metric, F.Cu at (128.0, 107.8)
- added C917: 4.7uF, Capacitor_SMD:C_0805_2012Metric, F.Cu at (125.2, 108.6)
- added D801: BLUE, LED_SMD:LED_0805_2012Metric, F.Cu at (96.7, 29.6)
- added D802: BLUE, LED_SMD:LED_0805_2012Metric, F.Cu at (119.1, 22.1)
- added D803: BLUE, LED_SMD:LED_0805_2012Metric, F.Cu at (119.1, 29.5)
- added D804: BLUE, LED_SMD:LED_0805_2012Metric, F.Cu at (139.3, 22.2)
- added D805: BLUE, LED_SMD:LED_0805_2012Metric, F.Cu at (139.3, 29.5)
- added D806: BLUE, LED_SMD:LED_0805_2012Metric, F.Cu at (75.2, 22.5)
- added D807: BLUE, LED_SMD:LED_0805_2012Metric, F.Cu at (75.2, 29.7)
- added D808: BLUE, LED_SMD:LED_0805_2012Metric, F.Cu at (96.7, 22.3)
- added D809: BLUE, LED_SMD:LED_0805_2012Metric, F.Cu at (96.7, 33.3)
- added D810: BLUE, LED_SMD:LED_0805_2012Metric, F.Cu at (119.1, 25.8)
- added D811: BLUE, LED_SMD:LED_0805_2012Metric, F.Cu at (119.1, 33.2)
- added D812: BLUE, LED_SMD:LED_0805_2012Metric, F.Cu at (139.3, 25.8)
- added D813: BLUE, LED_SMD:LED_0805_2012Metric, F.Cu at (139.3, 33.2)
- added D814: BLUE, LED_SMD:LED_0805_2012Metric, F.Cu at (75.2, 26.0)
- added D815: BLUE, LED_SMD:LED_0805_2012Metric, F.Cu at (75.2, 33.5)
- added D816: BLUE, LED_SMD:LED_0805_2012Metric, F.Cu at (96.7, 26.0)
- added D817: BLUE, LED_SMD:LED_0805_2012Metric, F.Cu at (160.0, 22.1)
- added D901: RED, LED_SMD:LED_0805_2012Metric, F.Cu at (126.5, 139.4)
- added D902: RED, LED_SMD:LED_0805_2012Metric, F.Cu at (126.4, 135.8)
- added D903: RED, LED_SMD:LED_0805_2012Metric, F.Cu at (126.4, 147.0)
- added D904: RED, LED_SMD:LED_0805_2012Metric, F.Cu at (126.4, 143.2)
- added F301: 16V/1.1A, Fuse:Fuse_1812_4532Metric, F.Cu at (79.1, 128.1)
- added FB601: 330R, Inductor_SMD:L_0805_2012Metric, B.Cu at (218.7, 135.8)
- added FB901: 120R, Inductor_SMD:L_0805_2012Metric, F.Cu at (123.2, 108.6)
- added J202: Screw_Terminal_01x02, TerminalBlock:TerminalBlock_bornier-2_P5.08mm, F.Cu at (99.3, 62.6)
- added J302: Screw_Terminal_01x02, TerminalBlock:TerminalBlock_bornier-2_P5.08mm, F.Cu at (79.1, 144.6)
- added J604: USB_A, Connector_USB:USB_A_Connfly_DS1095, F.Cu at (224.3, 132.8)
- added J605: RJ45_Hanrun_HR911105A_Horizontal, Connector_RJ:RJ45_Hanrun_HR911105A_Horizontal, F.Cu at (156.6, 135.6)
- added J901: RJ45_Hanrun_HR911105A_Horizontal, Connector_RJ:RJ45_Hanrun_HR911105A_Horizontal, F.Cu at (137.4, 135.6)
- added JP301: SolderJumper_2_Open, Jumper:SolderJumper-2_P1.3mm_Open_TrianglePad1.0x1.5mm, F.Cu at (87.5, 127.9)
- added Q301: DMT6007LFG, DMT6007LFG:DMP4013LFG7, F.Cu at (31.8, 100.7)
- added Q302: DMT6007LFG, DMT6007LFG:DMP4013LFG7, F.Cu at (31.7, 105.5)
- added Q303: SSM6K518NU, footprints:SOT-1220UDFN6B_TOS, F.Cu at (84.6, 132.1)
- added Q601: SSM6K518NU, footprints:SOT-1220UDFN6B_TOS, F.Cu at (200.7, 111.9)
- added Q801: BSS138 JI, Package_TO_SOT_SMD:SOT-23, B.Cu at (93.0, 29.6)
- added Q802: BSS138 JI, Package_TO_SOT_SMD:SOT-23, B.Cu at (115.3, 22.1)
- added Q803: BSS138 JI, Package_TO_SOT_SMD:SOT-23, B.Cu at (115.4, 29.5)
- added Q804: BSS138 JI, Package_TO_SOT_SMD:SOT-23, B.Cu at (135.6, 22.2)
- added Q805: BSS138 JI, Package_TO_SOT_SMD:SOT-23, B.Cu at (135.5, 29.5)
- added Q806: BSS138 JI, Package_TO_SOT_SMD:SOT-23, B.Cu at (71.5, 22.5)
- added Q807: BSS138 JI, Package_TO_SOT_SMD:SOT-23, B.Cu at (71.5, 29.7)
- added Q808: BSS138 JI, Package_TO_SOT_SMD:SOT-23, B.Cu at (93.0, 22.3)
- added Q809: BSS138 JI, Package_TO_SOT_SMD:SOT-23, B.Cu at (92.9, 33.3)
- added Q810: BSS138 JI, Package_TO_SOT_SMD:SOT-23, B.Cu at (115.3, 25.8)
- added Q811: BSS138 JI, Package_TO_SOT_SMD:SOT-23, B.Cu at (115.4, 33.2)
- added Q812: BSS138 JI, Package_TO_SOT_SMD:SOT-23, B.Cu at (135.6, 25.8)
- added Q813: BSS138 JI, Package_TO_SOT_SMD:SOT-23, B.Cu at (135.6, 33.2)
- added Q814: BSS138 JI, Package_TO_SOT_SMD:SOT-23, B.Cu at (71.5, 26.0)
- added Q815: BSS138 JI, Package_TO_SOT_SMD:SOT-23, B.Cu at (71.5, 33.5)
- added Q816: BSS138 JI, Package_TO_SOT_SMD:SOT-23, B.Cu at (93.0, 26.0)
- added Q817: BSS138 JI, Package_TO_SOT_SMD:SOT-23, B.Cu at (156.3, 22.1)
- added R219: 10K, Resistor_SMD:R_0805_2012Metric, F.Cu at (67.4, 84.8)
- added R220: 2mR, Resistor_SMD:R_2512_6332Metric, F.Cu at (71.9, 74.7)
- added R224: 10K, Resistor_SMD:R_0805_2012Metric, F.Cu at (67.4, 82.8)
- added R301: 10K, Resistor_SMD:R_0805_2012Metric, F.Cu at (68.1, 122.6)
- added R302: 10K, Resistor_SMD:R_0805_2012Metric, F.Cu at (68.1, 124.6)
- added R303: 2mR, Resistor_SMD:R_2512_6332Metric, F.Cu at (79.1, 118.2)
- added R308: 2mR, Resistor_SMD:R_2512_6332Metric, F.Cu at (61.8, 82.8)
- added R309: 10K, Resistor_SMD:R_0805_2012Metric, F.Cu at (87.3, 99.9)
- added R312: 10K, Resistor_SMD:R_0805_2012Metric, F.Cu at (87.3, 101.9)
- added R313: 10K, Resistor_SMD:R_0805_2012Metric, F.Cu at (87.3, 97.9)
- added R314: 2mR, Resistor_SMD:R_2512_6332Metric, F.Cu at (41.3, 130.2)
- added R317: 10K, Resistor_SMD:R_0805_2012Metric, F.Cu at (50.7, 139.5)
- added R319: 10K, Resistor_SMD:R_0805_2012Metric, F.Cu at (50.7, 141.5)
- added R320: 10K, Resistor_SMD:R_0805_2012Metric, F.Cu at (50.7, 137.5)
- added R723: 105R, Resistor_SMD:R_0805_2012Metric, F.Cu at (137.7, 49.2)
- added R724: 105R, Resistor_SMD:R_0805_2012Metric, F.Cu at (137.7, 54.4)
- added R725: 105R, Resistor_SMD:R_0805_2012Metric, F.Cu at (163.8, 39.0)
- added R730: 105R, Resistor_SMD:R_0805_2012Metric, F.Cu at (163.8, 44.0)
- added R731: 105R, Resistor_SMD:R_0805_2012Metric, F.Cu at (163.8, 49.2)
- added R733: 100K, Resistor_SMD:R_0805_2012Metric, F.Cu at (204.4, 43.3)
- added R736: 105R, Resistor_SMD:R_0805_2012Metric, F.Cu at (189.2, 39.0)
- added R737: 1K2, Resistor_SMD:R_1206_3216Metric, F.Cu at (189.3, 44.2)
- added R738: 1K2, Resistor_SMD:R_1206_3216Metric, F.Cu at (189.2, 49.2)
- added R801: 200R, Resistor_SMD:R_0805_2012Metric, B.Cu at (96.7, 29.6)
- added R802: 200R, Resistor_SMD:R_0805_2012Metric, B.Cu at (119.1, 22.1)
- added R803: 200R, Resistor_SMD:R_0805_2012Metric, B.Cu at (119.1, 29.5)
- added R804: 200R, Resistor_SMD:R_0805_2012Metric, B.Cu at (139.3, 22.2)
- added R805: 200R, Resistor_SMD:R_0805_2012Metric, B.Cu at (139.3, 29.5)
- added R806: 200R, Resistor_SMD:R_0805_2012Metric, B.Cu at (75.2, 22.5)
- added R807: 200R, Resistor_SMD:R_0805_2012Metric, B.Cu at (75.2, 29.7)
- added R808: 200R, Resistor_SMD:R_0805_2012Metric, B.Cu at (96.7, 22.3)
- added R809: 200R, Resistor_SMD:R_0805_2012Metric, B.Cu at (96.7, 33.3)
- added R810: 200R, Resistor_SMD:R_0805_2012Metric, B.Cu at (119.1, 25.8)
- added R811: 200R, Resistor_SMD:R_0805_2012Metric, B.Cu at (119.1, 33.2)
- added R812: 200R, Resistor_SMD:R_0805_2012Metric, B.Cu at (139.3, 25.8)
- added R813: 200R, Resistor_SMD:R_0805_2012Metric, B.Cu at (139.3, 33.2)
- added R814: 200R, Resistor_SMD:R_0805_2012Metric, B.Cu at (75.2, 26.0)
- added R815: 200R, Resistor_SMD:R_0805_2012Metric, B.Cu at (75.2, 33.5)
- added R816: 200R, Resistor_SMD:R_0805_2012Metric, B.Cu at (96.7, 26.0)
- added R817: 200R, Resistor_SMD:R_0805_2012Metric, B.Cu at (160.0, 22.1)
- added R901: 49R9, Resistor_SMD:R_0805_2012Metric, F.Cu at (115.3, 97.6)
- added R902: 49R9, Resistor_SMD:R_0805_2012Metric, B.Cu at (111.6, 100.7)
- added R903: 10R, Resistor_SMD:R_0805_2012Metric, F.Cu at (111.2, 97.0)
- added R904: 330R, Resistor_SMD:R_0805_2012Metric, F.Cu at (125.6, 87.0)
- added R905: 330R, Resistor_SMD:R_0805_2012Metric, F.Cu at (122.2, 87.0)
- added R906: 10K, Resistor_SMD:R_0805_2012Metric, B.Cu at (127.3, 101.2)
- added R907: 0R, Resistor_SMD:R_0805_2012Metric, B.Cu at (115.3, 97.6)
- added R908: 0R, Resistor_SMD:R_0805_2012Metric, B.Cu at (115.3, 99.5)
- added R909: 330R, Resistor_SMD:R_0805_2012Metric, B.Cu at (146.9, 144.7)
- added R910: 330R, Resistor_SMD:R_0805_2012Metric, F.Cu at (125.6, 89.0)
- added R911: 330R, Resistor_SMD:R_0805_2012Metric, F.Cu at (122.2, 89.0)
- added R912: 0R, Resistor_SMD:R_0805_2012Metric, F.Cu at (115.3, 99.5)
- added R913: 10K, Resistor_SMD:R_0805_2012Metric, F.Cu at (128.2, 93.8)
- added R914: 0R, Resistor_SMD:R_0805_2012Metric, F.Cu at (115.3, 101.5)
- added R915: 330R, Resistor_SMD:R_0805_2012Metric, B.Cu at (136.9, 144.7)
- added R916: 330R, Resistor_SMD:R_0805_2012Metric, F.Cu at (125.6, 91.0)
- added R917: 330R, Resistor_SMD:R_0805_2012Metric, F.Cu at (122.2, 91.0)
- added R918: 82R, Resistor_SMD:R_0805_2012Metric, F.Cu at (110.1, 105.2)
- added R919: 82R, Resistor_SMD:R_0805_2012Metric, F.Cu at (107.5, 105.2)
- added R920: 1M, Resistor_SMD:R_0805_2012Metric, B.Cu at (131.4, 101.8)
- added R921: 130R, Resistor_SMD:R_0805_2012Metric, F.Cu at (129.8, 139.4)
- added R922: 130R, Resistor_SMD:R_0805_2012Metric, F.Cu at (129.8, 135.8)
- added R923: 12.4K 1%, Resistor_SMD:R_0805_2012Metric, F.Cu at (119.2, 106.1)
- added R924: 130R, Resistor_SMD:R_0805_2012Metric, F.Cu at (129.9, 147.0)
- added R925: 130R, Resistor_SMD:R_0805_2012Metric, F.Cu at (129.9, 143.2)
- added U301: INA226, Package_SO:VSSOP-10_3x3mm_P0.5mm, F.Cu at (73.4, 122.8)
- added U303: LM74700QDDFRQ1, LM74700QDDFRQ1:SOT65P280X110-8N, F.Cu at (27.5, 100.8)
- added U304: TVS2701DRBR, TVS2701DRBR:IC_TVS2701DRBR, F.Cu at (20.4, 101.0)
- added U306: INA226, Package_SO:VSSOP-10_3x3mm_P0.5mm, F.Cu at (92.5, 99.8)
- added U307: LM74700QDDFRQ1, LM74700QDDFRQ1:SOT65P280X110-8N, F.Cu at (27.4, 105.6)
- added U308: TVS2701DRBR, TVS2701DRBR:IC_TVS2701DRBR, F.Cu at (20.3, 105.3)
- added U310: INA226, Package_SO:VSSOP-10_3x3mm_P0.5mm, F.Cu at (55.9, 139.1)
- added U311: LM74700QDDFRQ1, LM74700QDDFRQ1:SOT65P280X110-8N, F.Cu at (84.5, 127.9)
- added U603: USBLC6-2SC6, Package_TO_SOT_SMD:SOT-23-6, B.Cu at (219.8, 129.3)
- added U708: 74LVC1G14GW-Q100,1, Package_TO_SOT_SMD:SOT-353_SC-70-5, F.Cu at (209.2, 49.0)
- added U901: W5500, Package_QFP:LQFP-48_7x7mm_P0.5mm, F.Cu at (124.6, 101.0)
- added Y901: 25MHz, Crystal:Crystal_SMD_3225-4Pin_3.2x2.5mm, F.Cu at (132.2, 102.0)
- C301: value 330uF 25V -> 0.1uF; footprint Capacitor_SMD:CP_Elec_8x10.5 -> Capacitor_SMD:C_0805_2012Metric
- C401: value 100nF -> 1uF
- C402: value 22pF -> 1uF
- C403: value 22pF -> 100nF; footprint Capacitor_SMD:C_0805_2012Metric -> Capacitor_SMD:C_1206_3216Metric
- C601: value 10uF -> 100nF; footprint Capacitor_Tantalum_SMD:CP_EIA-3216-10_Kemet-I -> Capacitor_SMD:C_1206_3216Metric
- C602: moved to B.Cu
- C604: renamed from C603; moved to B.Cu
- C701: renamed from C714; value 47uF -> 1uF; moved to B.Cu
- C704: renamed from C715; value 47uF -> 1uF; moved to B.Cu
- C711: renamed from C716; value 47uF -> 1uF; moved to B.Cu
- C718, C719: value 47uF -> 1uF
- D201: footprint LED_SMD:LED_1210_3225Metric -> LED_SMD:LED_0805_2012Metric
- D202: renamed from D209; footprint LED_SMD:LED_1210_3225Metric -> LED_SMD:LED_0805_2012Metric
- D203: renamed from D217; footprint LED_SMD:LED_1210_3225Metric -> LED_SMD:LED_0805_2012Metric
- D204: renamed from D202; moved to B.Cu
- D205: renamed from D210; moved to B.Cu
- D206: renamed from D218; moved to B.Cu
- D207: renamed from D203; footprint LED_SMD:LED_1210_3225Metric -> LED_SMD:LED_0805_2012Metric
- D208: renamed from D211; footprint LED_SMD:LED_1210_3225Metric -> LED_SMD:LED_0805_2012Metric
- D209: renamed from D219; footprint LED_SMD:LED_1210_3225Metric -> LED_SMD:LED_0805_2012Metric
- D210: renamed from D204; moved to B.Cu
- D211: renamed from D212; moved to B.Cu
- D212: renamed from D220; moved to B.Cu
- D213: renamed from D205; footprint LED_SMD:LED_1210_3225Metric -> LED_SMD:LED_0805_2012Metric
- D214: renamed from D213; footprint LED_SMD:LED_1210_3225Metric -> LED_SMD:LED_0805_2012Metric
- D215: renamed from D206; moved to B.Cu
- D216: renamed from D214; moved to B.Cu
- D217: renamed from D207; footprint LED_SMD:LED_1210_3225Metric -> LED_SMD:LED_0805_2012Metric
- D218: renamed from D215; footprint LED_SMD:LED_1210_3225Metric -> LED_SMD:LED_0805_2012Metric
- D219: renamed from D208; moved to B.Cu
- D220: renamed from D216; moved to B.Cu
- D302: renamed from D303; footprint LED_SMD:LED_1210_3225Metric -> LED_SMD:LED_0805_2012Metric
- F201: value 500mA -> 3512P; footprint Fuse:Fuse_1812_4532Metric -> Fuse:Fuseholder_Clip-5x20mm_Keystone_3512P_Inline_P23.62x7.27mm_D1.02x2.41x1.02x1.57mm_Horizontal
- F601: footprint Fuse:Fuse_1812_4532Metric -> Fuse:Fuse_0805_2012Metric; moved to B.Cu
- JP401: value Jumper_2_Open -> SolderJumper_2_Open; footprint TestPoint:TestPoint_2Pads_Pitch2.54mm_Drill0.8mm -> Jumper:SolderJumper-2_P1.3mm_Open_TrianglePad1.0x1.5mm
- JP601: value Jumper_2_Bridged -> SolderJumper_2_Open; footprint TestPoint:TestPoint_2Pads_Pitch2.54mm_Drill0.8mm -> Jumper:SolderJumper-2_P1.3mm_Open_TrianglePad1.0x1.5mm
- Q401: value DMP3099L -> SSM6K518NU; footprint Package_TO_SOT_SMD:SOT-23-3 -> footprints:SOT-1220UDFN6B_TOS
- R201: renamed from R205; footprint Resistor_SMD:R_1206_3216Metric -> Resistor_SMD:R_0805_2012Metric
- R202: renamed from R213; footprint Resistor_SMD:R_1206_3216Metric -> Resistor_SMD:R_0805_2012Metric
- R203: renamed from R219; footprint Resistor_SMD:R_1206_3216Metric -> Resistor_SMD:R_0805_2012Metric
- R204: renamed from R201; footprint Resistor_SMD:R_1206_3216Metric -> Resistor_SMD:R_0805_2012Metric; moved to B.Cu
- R205: renamed from R209; footprint Resistor_SMD:R_1206_3216Metric -> Resistor_SMD:R_0805_2012Metric; moved to B.Cu
- R206: renamed from R217; footprint Resistor_SMD:R_1206_3216Metric -> Resistor_SMD:R_0805_2012Metric; moved to B.Cu
- R207: renamed from R206; footprint Resistor_SMD:R_1206_3216Metric -> Resistor_SMD:R_0805_2012Metric
- R208: renamed from R214; footprint Resistor_SMD:R_1206_3216Metric -> Resistor_SMD:R_0805_2012Metric
- R209: renamed from R220; footprint Resistor_SMD:R_1206_3216Metric -> Resistor_SMD:R_0805_2012Metric
- R210: renamed from R202; footprint Resistor_SMD:R_1206_3216Metric -> Resistor_SMD:R_0805_2012Metric; moved to B.Cu
- R211: renamed from R210; footprint Resistor_SMD:R_1206_3216Metric -> Resistor_SMD:R_0805_2012Metric; moved to B.Cu
- R212: renamed from R218; footprint Resistor_SMD:R_1206_3216Metric -> Resistor_SMD:R_0805_2012Metric; moved to B.Cu
- R213: renamed from R207; footprint Resistor_SMD:R_1206_3216Metric -> Resistor_SMD:R_0805_2012Metric
- R214: renamed from R215; footprint Resistor_SMD:R_1206_3216Metric -> Resistor_SMD:R_0805_2012Metric
- R215: renamed from R203; footprint Resistor_SMD:R_1206_3216Metric -> Resistor_SMD:R_0805_2012Metric; moved to B.Cu
- R216: renamed from R211; footprint Resistor_SMD:R_1206_3216Metric -> Resistor_SMD:R_0805_2012Metric; moved to B.Cu
- R217: renamed from R208; footprint Resistor_SMD:R_1206_3216Metric -> Resistor_SMD:R_0805_2012Metric
- R218: renamed from R216; footprint Resistor_SMD:R_1206_3216Metric -> Resistor_SMD:R_0805_2012Metric
- R221: value 5K1 -> 10K
- R222: renamed from R204; footprint Resistor_SMD:R_1206_3216Metric -> Resistor_SMD:R_0805_2012Metric; moved to B.Cu
- R223: renamed from R212; footprint Resistor_SMD:R_1206_3216Metric -> Resistor_SMD:R_0805_2012Metric; moved to B.Cu
- R304: value 200R -> 10K; footprint Resistor_SMD:R_1206_3216Metric -> Resistor_SMD:R_0805_2012Metric
- R307: renamed from R301; footprint Resistor_SMD:R_1206_3216Metric -> Resistor_SMD:R_0805_2012Metric
- R401: renamed from R407; value 4K7 -> 10K
- R402: renamed from R408; value 4K7 -> 10K
- R404: value 1K -> 10K
- R603: renamed from R605; moved to B.Cu
- R605: renamed from R606; moved to B.Cu
- R701, R702, R703, R709, R712, R713, R714: value 1K2 -> 105R
- R708: renamed from R704; value 1K2 -> 105R
- R719, R720, R735: value 200R -> 105R; footprint Resistor_SMD:R_1206_3216Metric -> Resistor_SMD:R_0805_2012Metric
- R734: value 200R -> 100K; footprint Resistor_SMD:R_1206_3216Metric -> Resistor_SMD:R_0805_2012Metric
- U201: value USBLC6-2SC6 -> INA226; footprint Package_TO_SOT_SMD:SOT-23-6 -> Package_SO:VSSOP-10_3x3mm_P0.5mm
- U402: value SN74LVC1G125DCK -> NC7SZ08M5X; footprint Package_TO_SOT_SMD:Texas_R-PDSO-G5_DCK-5 -> Package_TO_SOT_SMD:SOT-23-5
- U403: value SN74LVC1G125DCK -> APX811-31UG-7; footprint Package_TO_SOT_SMD:Texas_R-PDSO-G5_DCK-5 -> Package_TO_SOT_SMD:SOT-143
- U404: value ATSAM3X8EA-AU -> LM74700QDDFRQ1; footprint ATSAM3X8EA-AU:QFP50P2200X2200X145-144N -> LM74700QDDFRQ1:SOT65P280X110-8N
- U601: value USBLC6-2SC6 -> LM74700QDDFRQ1; footprint Package_TO_SOT_SMD:SOT-23-6 -> LM74700QDDFRQ1:SOT65P280X110-8N; moved to F.Cu
- U702: renamed from U701; moved to B.Cu
- U704: renamed from U702; moved to B.Cu
- U706: renamed from U703; moved to B.Cu
- moved R603 117.6 mm to (166.8, 144.8)
- moved C605 115.9 mm to (234.3, 40.3), turned to 180 degrees
- moved R606 114.9 mm to (234.3, 42.3), turned to 0 degrees
- moved SW601 112.7 mm to (234.3, 47.8), turned to -90 degrees
- moved R605 112.0 mm to (155.4, 144.8), turned to 0 degrees
- moved C604 102.0 mm to (162.0, 129.2), turned to 90 degrees
- moved C602 99.6 mm to (160.0, 129.2), turned to 90 degrees
- moved R214 95.5 mm to (24.0, 76.5), turned to 90 degrees
- moved D214 93.8 mm to (24.0, 73.6), turned to -90 degrees
- moved R404 93.1 mm to (173.6, 74.5), turned to 180 degrees
- moved R403 92.8 mm to (169.4, 74.5), turned to 180 degrees
- moved R734 88.6 mm to (204.4, 48.2), turned to -90 degrees
- moved R218 82.8 mm to (36.0, 76.5), turned to 90 degrees
- moved D218 81.0 mm to (36.0, 73.5), turned to -90 degrees
- moved J601 79.3 mm to (220.6, 37.5)
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- renumbered C304 to C302, C307 to C303, C303 to C308, C305 to C309, C306 to C313, C308 to C314, C607 to C605, C701 to C702, C706 to C703, C702 to C705, C707 to C706, C711 to C707, C713 to C708, C703 to C709, C708 to C710, C704 to C712, C709 to C713, C710 to C714, C712 to C715, C705 to C717, D308 to D301, D306 to D303, D310 to D304, H103 to H102, H102 to H103, J202 to J201, J605 to J601, J604 to J602, Q205 to Q202, Q209 to Q203, Q202 to Q204, Q206 to Q205, Q210 to Q206, Q203 to Q207, Q207 to Q208, Q204 to Q209, Q208 to Q210, Q601 to Q602, R302 to R310, R303 to R311, R308 to R315, R309 to R316, R310 to R318, R445 to R405, R444 to R406, R608 to R601, R609 to R602, R610 to R604, R607 to R606, R723 to R704, R730 to R705, R736 to R706, R742 to R707, R724 to R710, R729 to R711, R725 to R715, R731 to R716, R738 to R717, R743 to R718, R726 to R721, R732 to R722, R727 to R726, R733 to R727, R737 to R728, R739 to R729, R728 to R732, U301 to U305, U303 to U309, IC401 to U401, U603 to U602, IC701 to U701, IC702 to U703, IC703 to U705, IC704 to U707, IC705 to U709
Connections:
- net /ATMEL SAM3X8/FEED_FORWARD renamed /Arduino Due/D26/PIN26
- net /ATMEL SAM3X8/FEED_REVERSE renamed /Arduino Due/D27/PIN27
- net /ATMEL SAM3X8/HEAD_CCW renamed /Arduino Due/D29/PIN29
- net /ATMEL SAM3X8/HEAD_CW renamed /Arduino Due/D28/PIN28
- net /ATMEL SAM3X8/HEAD_IN renamed /Arduino Due/D31/PIN31
- net /ATMEL SAM3X8/HEAD_OUT renamed /Arduino Due/D30/PIN30
- net /ATMEL SAM3X8/SHEAR_CUT renamed /Arduino Due/D22/PIN22
- net /ATMEL SAM3X8/SHEAR_HOME renamed /Arduino Due/D23/PIN23
- net /ATMEL SAM3X8/TOOL_IN renamed /Arduino Due/D25/PIN25
- net /ATMEL SAM3X8/TOOL_OUT renamed /Arduino Due/D24/PIN24
- net /Pi Zero 2W SBC/PI13 renamed /Pi Zero 2W SBC/PWM/UART4_TX
- net /Signal Processing/AUTO_BUTTON renamed /Input Connections/AUTO_BUTTON
- net /Signal Processing/ENCODER_BEND_RESET renamed /Input Connections/ENCODER_BEND_RESET
- net /Signal Processing/ENCODER_BEND_SET renamed /Input Connections/ENCODER_BEND_SET
- net /Signal Processing/ENCODER_FEED_RESET renamed /Input Connections/ENCODER_FEED_RESET
- net /Signal Processing/ENCODER_FEED_SET renamed /Input Connections/ENCODER_FEED_SET
- net /Signal Processing/PROXIMITY_HEAD_CCW renamed /Input Connections/PROXIMITY_HEAD_CCW
- net /Signal Processing/PROXIMITY_HEAD_CW renamed /Input Connections/PROXIMITY_HEAD_CW
- net /Signal Processing/PROXIMITY_HEAD_IN renamed /Input Connections/PROXIMITY_HEAD_IN
- net /Signal Processing/PROXIMITY_HEAD_LIM renamed /Input Connections/PROXIMITY_HEAD_LIM
- net /Signal Processing/PROXIMITY_HEAD_OUT renamed /Input Connections/PROXIMITY_HEAD_OUT
- net /Signal Processing/PROXIMITY_SHEAR_CUT renamed /Input Connections/PROXIMITY_SHEAR_CUT
- net /Signal Processing/PROXIMITY_SHEAR_HOME renamed /Input Connections/PROXIMITY_SHEAR_HOME
- net /Signal Processing/PROXIMITY_TOOL_IN renamed /Input Connections/PROXIMITY_TOOL_IN
- net /Signal Processing/PROXIMITY_TOOL_OUT renamed /Input Connections/PROXIMITY_TOOL_OUT
- net /Signal Processing/SHEAR_BUTTON renamed /Input Connections/SHEAR_BUTTON
- net /Signal Processing/~{ESTOP} renamed /Arduino Due/D47/PIN47
- C301 pad 1: Net-(D303-A) -> GND
- C301 pad 2: GND -> +3V3
- C303 pad 1: +12V -> /External Power/12VOUT
- C309 pad 1: +5V -> /External Power/5VOUT
- C314 pad 1: +3V3 -> /External Power/3V3OUT
- C401 pad 1: +5V -> GND
- C401 pad 2: GND -> +3V3
- C402 pad 1: /ATMEL SAM3X8/XTAL1 -> GND
- C402 pad 2: GND -> +3V3
- C403 pad 1: /ATMEL SAM3X8/XTAL2 -> +12V
- C403 pad 2: GND -> Net-(U404-VCAP)
- C601 pad 1: +3V3 -> +5V
- C601 pad 2: GND -> Net-(U601-VCAP)
- C718 pad 1: GND -> /Signal Processing/24VRAW*
- C718 pad 2: +3V3 -> GND
- C719 pad 1: GND -> /Signal Processing/AUX24V*
- C719 pad 2: +3V3 -> GND
- D301 pad 2: +12V -> /External Power/12VOUT
- D302 pad 2: Net-(D303-A) -> +24V
- D303 pad 2: +5V -> /External Power/5VOUT
- D304 pad 2: +3V3 -> /External Power/3V3OUT
- F201 pad 1: /Output Connections/VUSB -> /Output Connections/FUSE
- F201 pad 2: /ATMEL SAM3X8/VUSBVCC -> /Output Connections/ESTOP
- F601 pad 1: /Pi Zero 2W SBC/VUSB -> Net-(J604-VBUS)
- F601 pad 2: /Pi Zero 2W SBC/VUSB-FUSED -> Net-(U603-VBUS)
- J301 pad 1: Net-(D301-A) -> AUX24V
- J601 pad 4: /Output Connections/SBC-USB2-D- -> /Pi Zero 2W SBC/USB2-D-
- J601 pad 5: /Output Connections/SBC-USB2-D+ -> /Pi Zero 2W SBC/USB2-D+
- J603 pad 8: +5V -> /Pi Zero 2W SBC/5V
- JP401 pad 1: /ATMEL SAM3X8/RXD1-16U2 -> +12V
- JP401 pad 2: /ATMEL SAM3X8/TX -> /Arduino Due/VIN
- JP601 pad 1: /Pi Zero 2W SBC/~{CTS} -> +5V
- JP601 pad 2: Net-(JP601-B) -> /Pi Zero 2W SBC/5V
- Q401 pad 1: /ATMEL SAM3X8/ERASE_CMD -> +12V
- Q401 pad 2: +3V3 -> Net-(Q401-G)
- Q401 pad 3: Net-(Q401-D) -> /Arduino Due/VIN
- Q602 pad 3: /ATMEL SAM3X8/MASTER-RESET -> /Arduino Due/~{ATSAM3X8E_RESET}
- R221 pad 1: GND -> +3V3
- R221 pad 2: Net-(J201-CC1) -> SCL
- R304 pad 1: GND -> +3V3
- R304 pad 2: Net-(D307-K) -> /Arduino Due/D51/PIN51
- R305 pad 1: +12V -> /External Power/12VOUT
- R310 pad 1: +5V -> /External Power/5VOUT
- R315 pad 1: +3V3 -> /External Power/3V3OUT
- R403 pad 1: GND -> SDA
- R403 pad 2: /ATMEL SAM3X8/USB_BOOT_EN -> +3V3
- R404 pad 1: /ATMEL SAM3X8/RESET_CMD -> +3V3
- R404 pad 2: /ATMEL SAM3X8/MASTER-RESET -> SCL
- R405 pad 1: SCL -> /Arduino Due/HMI_I2C_SDA1
- R406 pad 2: SDA -> /Arduino Due/HMI_I2C_SCL1
- R601 pad 1: SDA -> /Arduino Due/HMI_I2C_SDA1
- R602 pad 2: SCL -> /Arduino Due/HMI_I2C_SCL1
- R701 pad 1: +24V -> +3V3
- R702 pad 1: +24V -> +3V3
- R703 pad 1: +24V -> +3V3
- R708 pad 1: +24V -> +3V3
- R709 pad 1: +24V -> +3V3
- R709 pad 2: Net-(IC703-A_1) -> Net-(U703-A1)
- R712 pad 1: +24V -> +3V3
- R712 pad 2: Net-(IC703-A_4) -> Net-(U703-A2)
- R713 pad 1: +24V -> +3V3
- R713 pad 2: Net-(IC704-A_1) -> Net-(U703-A3)
- R714 pad 1: +24V -> +3V3
- R714 pad 2: Net-(IC704-A_2) -> Net-(U703-A4)
- R719 pad 1: Net-(D702-A) -> +3V3
- R719 pad 2: +5V -> Net-(U705-A1)
- R720 pad 1: Net-(D703-A) -> +3V3
- R720 pad 2: +5V -> Net-(U705-A2)
- R734 pad 1: Net-(D706-A) -> +3V3
- R734 pad 2: +5V -> /Signal Processing/AUX24V*
- R735 pad 1: Net-(D707-A) -> +3V3
- R735 pad 2: +5V -> Net-(U707-A4)
- U201 pad 1: /Output Connections/2D+ -> GND
- U201 pad 3: /Output Connections/2D- -> /Arduino Due/D13/PIN13
- U201 pad 4: /Output Connections/USBC-D- -> SDA
- U201 pad 5: /ATMEL SAM3X8/VUSBVCC -> SCL
- U201 pad 6: /Output Connections/USBC-D+ -> +3V3
- U302 pad 2: +12V -> /External Power/12VOUT
- U305 pad 2: +5V -> /External Power/5VOUT
- U309 pad 2: +3V3 -> /External Power/3V3OUT
- U402 pad 1: /ATMEL SAM3X8/TX -> /Arduino Due/D12/PIN12
- U402 pad 2: /ATMEL SAM3X8/TX -> /Arduino Due/~{ATSAM3X8E_RESET}
- U402 pad 4: /ATMEL SAM3X8/RXD1-16U2 -> Net-(U403-~{MR})
- U402 pad 5: +5V -> +3V3
- U403 pad 1: /ATMEL SAM3X8/TXD1-16U2 -> GND
- U403 pad 2: /ATMEL SAM3X8/TXD1-16U2 -> /Arduino Due/~{W5500_RST}
- U403 pad 3: GND -> Net-(U403-~{MR})
- U403 pad 4: /ATMEL SAM3X8/RX -> +3V3
- U404 pad 1: /ATMEL SAM3X8/D22/PIN22 -> +12V
- U404 pad 2: /ATMEL SAM3X8/TX -> GND
- U404 pad 3: /ATMEL SAM3X8/RXD2 -> unconnected-(U404-NC-Pad3)
- U404 pad 4: /ATMEL SAM3X8/TXD2 -> Net-(U404-VCAP)
- U404 pad 5: /ATMEL SAM3X8/RXD1 -> +12V
- U404 pad 6: /ATMEL SAM3X8/TXD1 -> Net-(Q401-G)
- U404 pad 7: /ATMEL SAM3X8/D23/PIN23 -> unconnected-(U404-NC-Pad7)
- U404 pad 8: /ATMEL SAM3X8/D24/PIN24 -> /Arduino Due/VIN
- U601 pad 1: /Pi Zero 2W SBC/2D+ -> +5V
- U601 pad 3: /Pi Zero 2W SBC/2D- -> unconnected-(U601-NC-Pad3)
- U601 pad 4: /Pi Zero 2W SBC/D- -> Net-(U601-VCAP)
- U601 pad 5: /Pi Zero 2W SBC/VUSB-FUSED -> +5V
- U601 pad 6: /Pi Zero 2W SBC/D+ -> Net-(Q601-G)
- U602 pad 11: /ATMEL SAM3X8/RXD1 -> /Arduino Due/HMI_UART_RX2
- U602 pad 13: /ATMEL SAM3X8/TXD1 -> /Arduino Due/HMI_UART_TX2
- U602 pad 15: /ATMEL SAM3X8/SCL1 -> /Arduino Due/HMI_UART_RX1
- U602 pad 19: /ATMEL SAM3X8/MOSI -> /Arduino Due/SPI_MOSI
- U602 pad 2: Net-(U603-5V_2) -> /Pi Zero 2W SBC/5V
- U602 pad 21: /ATMEL SAM3X8/MISO -> /Arduino Due/SPI_MISO
- U602 pad 22: /ATMEL SAM3X8/SDA1 -> /Arduino Due/HMI_UART_TX1
- U602 pad 23: /ATMEL SAM3X8/SPCK -> /Arduino Due/SPI_SCK
- U602 pad 24: /ATMEL SAM3X8/SPI1_CS0 -> /Arduino Due/D4_CS1/PIN4
- U602 pad 3: SDA -> /Arduino Due/HMI_I2C_SDA1
- U602 pad 32: /Pi Zero 2W SBC/PWM1 -> unconnected-(U602-GPIO12-Pad32)
- U602 pad 4: Net-(U603-5V_2) -> /Pi Zero 2W SBC/5V
- U602 pad 5: SCL -> /Arduino Due/HMI_I2C_SCL1
- U702 pad 10: /Signal Processing/~{PROXIMITY_HEAD_OUT} -> /Arduino Due/D36/PIN36
- U702 pad 12: /Signal Processing/~{PROXIMITY_HEAD_IN} -> /Arduino Due/D37/PIN37
- U702 pad 2: /Signal Processing/~{ENCODER_FEED_SET} -> /Arduino Due/D32/PIN32
- U702 pad 4: /Signal Processing/~{ENCODER_FEED_RESET} -> /Arduino Due/D33/PIN33
- U702 pad 6: /Signal Processing/~{ENCODER_BEND_SET} -> /Arduino Due/D34/PIN34
- U702 pad 8: /Signal Processing/~{ENCODER_BEND_RESET} -> /Arduino Due/D35/PIN35
- U703 pad 1: Net-(IC702-A_1) -> Net-(U703-A1)
- U703 pad 3: Net-(IC702-A_2) -> Net-(U703-A2)
- U703 pad 5: Net-(IC702-A_3) -> Net-(U703-A3)
- U703 pad 7: Net-(IC702-A_4) -> Net-(U703-A4)
- U704 pad 10: /Signal Processing/~{SHEAR_BUTTON} -> /Arduino Due/D42/PIN42
- U704 pad 12: /Signal Processing/~{PROXIMITY_HEAD_LIM} -> /Arduino Due/D43/PIN43
- U704 pad 2: /Signal Processing/~{PROXIMITY_SHEAR_HOME} -> /Arduino Due/D38/PIN38
- U704 pad 4: /Signal Processing/~{PROXIMITY_SHEAR_CUT} -> /Arduino Due/D39/PIN39
- U704 pad 6: /Signal Processing/~{PROXIMITY_TOOL_IN} -> /Arduino Due/D40/PIN40
- U704 pad 8: /Signal Processing/~{PROXIMITY_TOOL_OUT} -> /Arduino Due/D41/PIN41
- U705 pad 1: Net-(IC703-A_1) -> Net-(U705-A1)
- U705 pad 3: Net-(IC703-A_2) -> Net-(U705-A2)
- U705 pad 7: Net-(IC703-A_4) -> Net-(U705-A4)
- U706 pad 10: /Signal Processing/~{FUSE} -> /Arduino Due/D48/PIN48
- U706 pad 12: unconnected-(U703-6Y-Pad12) -> /Arduino Due/D49/PIN49
- U706 pad 13: GND -> /Signal Processing/24VRAW*
- U706 pad 2: /Signal Processing/~{PROXIMITY_HEAD_CW} -> /Arduino Due/D44/PIN44
- U706 pad 4: /Signal Processing/~{PROXIMITY_HEAD_CCW} -> /Arduino Due/D45/PIN45
- U706 pad 6: /Signal Processing/~{AUTO_BUTTON} -> /Arduino Due/D46/PIN46
- U707 pad 1: Net-(IC704-A_1) -> Net-(U707-A1)
- U707 pad 3: Net-(IC704-A_2) -> Net-(U707-A2)
- U707 pad 7: Net-(IC704-A_4) -> Net-(U707-A4)
- U707 pad 8: /Signal Processing/ESTOP -> /Output Connections/ESTOP
- U709 pad 11: unconnected-(IC705-E_3-Pad11) -> GND
- U709 pad 12: unconnected-(IC705-C_3-Pad12) -> /Signal Processing/AUX24V*
- U709 pad 13: unconnected-(IC705-E_2-Pad13) -> GND
- U709 pad 14: unconnected-(IC705-C-2-Pad14) -> /Signal Processing/24VRAW*
- U709 pad 2: /Output Connections/FUSED_GND -> /Output Connections/FUSE
- U709 pad 3: unconnected-(IC705-A_2-Pad3) -> Net-(U709-A2)
- U709 pad 4: unconnected-(IC705-K_2-Pad4) -> GND
- U709 pad 5: unconnected-(IC705-A_3-Pad5) -> Net-(U709-A3)
- U709 pad 6: unconnected-(IC705-K_3-Pad6) -> GND
Routing:
- net /Output Connections/FUSED_GND: track 485.2 -> 14.0 mm, vias 23 -> 10
- net AUX24V: track 0.00 -> 420.9 mm, vias 0 -> 1
- net +3V3: track 636.8 -> 973.8 mm, vias 55 -> 72
- net /ATMEL SAM3X8/MASTER-RESET: track 283.7 -> 0.00 mm
- net +24V: track 292.6 -> 71.6 mm, vias 19 -> 0
- net /Output Connections/SBC-USB2-D+: track 216.2 -> 0.00 mm, vias 2 -> 0
- net /Arduino Due/~{ATSAM3X8E_RESET}: track 0.00 -> 216.2 mm, vias 0 -> 2
- net /Output Connections/SBC-USB2-D-: track 213.6 -> 0.00 mm, vias 2 -> 0
- net /Arduino Due/D35/PIN35: track 0.00 -> 204.5 mm, vias 0 -> 9
- net /Arduino Due/D33/PIN33: track 0.00 -> 194.6 mm, vias 0 -> 3
- net /Arduino Due/D40/PIN40: track 0.00 -> 189.2 mm, vias 0 -> 1
- net /Arduino Due/D39/PIN39: track 0.00 -> 188.4 mm, vias 0 -> 5
- net /Output Connections/FUSE: track 0.00 -> 187.0 mm
- net /Arduino Due/D45/PIN45: track 0.00 -> 181.1 mm, vias 0 -> 1
- net /Arduino Due/D37/PIN37: track 0.00 -> 178.8 mm, vias 0 -> 5
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- added copper zone on In2.Cu, net +12V
- added copper zone on F.Cu, net /Arduino Due/VIN
- added copper zone on F.Cu, net /External Power/+12V-HMI-FUSED
- added copper zone on F.Cu, net /External Power/12V
- added copper zone on F.Cu, net /External Power/12VOUT
- added copper zone on F.Cu, net /External Power/3V3OUT
- added copper zone on F.Cu, net /External Power/5VOUT
- added copper zone on F.Cu, net /Output Connections/ESTOP
- added copper zone on F.Cu, net /Output Connections/FUSE
- added copper zone on F.Cu, net /Pi Zero 2W SBC/5V
- added copper zone on B.Cu, net 24VRAW
- added copper zone on F.Cu, net 24VRAW
- added copper zone on In1.Cu, net 24VRAW
- added copper zone on In2.Cu, net 24VRAW
- added copper zone on F.Cu, net AUX24V
- added copper zone on B.Cu, net Net-(U709-A2)
- added copper zone on F.Cu, net Net-(U709-A2)
- added copper zone on In1.Cu, net Net-(U709-A2)
- added copper zone on In2.Cu, net Net-(U709-A2)
- added copper zone on F.Cu, net Net-(U709-A3)
- removed copper zone on F.Cu, net +3V3
- removed copper zone on In2.Cu, net +3V3
- removed copper zone on F.Cu, net /Signal Processing/ESTOP
- removed copper zone on F.Cu, net Net-(D301-A)
- removed copper zone on F.Cu, net Net-(D301-K)
- removed copper zone on F.Cu, net Net-(D303-A)
- removed copper zone on F.Cu, net Net-(D602-K)
- removed copper zone on F.Cu, net Net-(U603-5V_2)
Other:
- board text added: "+12V 1.1A"
- board text added: "100Mbps"
- board text added: "10Mbps"
- board text added: "AUX24V"
- board text added: "Full-duplex"
- board text added: "Half-duplex"
- board text added: "Interface Board Hardware: Connor McMillan Firmware: John Gilcreast Rev X3"
- board text added: "PI02W PWR"
- board text added: "PI02W USB"
- board text removed: "+12V 5A"
- board text removed: "24V"
- board text removed: "AB"
- board text removed: "AB*"
- board text removed: "E"
- board text removed: "E*"
- board text removed: "EBR"
- board text removed: "EBR*"
- board text removed: "EBS"
- board text removed: "EBS*"
- board text removed: "EFR"
- board text removed: "EFR*"
- board text removed: "EFS"
- board text removed: "EFS*"
- board text removed: "F"
- board text removed: "F*"
- board text removed: "FG"
- board text removed: "Interface Board Hardware: Connor McMillan Firmware: John Gilcreast Rev X2"
- board text removed: "PHC"
- board text removed: "PHC*"
- board text removed: "PHCC"
- board text removed: "PHCC*"
- board text removed: "PHI"
- board text removed: "PHI*"
- board text removed: "PHL"
- board text removed: "PHL*"
- board text removed: "PHO"
- board text removed: "PHO*"
- board text removed: "PI 0 2W DEBUG"
- board text removed: "PI 0 2W PWR"
- board text removed: "PSC"
- board text removed: "PSC*"
- board text removed: "PSH"
- board text removed: "PSH*"
- board text removed: "PTI"
- board text removed: "PTI*"
- board text removed: "PTO"
- board text removed: "PTO*"
- board text removed: "RESET"
- board text removed: "RX"
- board text removed: "SAM3X8"
- board text removed: "SB"
- board text removed: "SB*"
- board text removed: "SBC"
- board text removed: "TX"
- board text removed: "USBC"
- board text removed: "~{AB}"
- board text removed: "~{EBR}"
- board text removed: "~{EBS}"
- board text removed: "~{EFR}"
- board text removed: "~{EFS}"
- board text removed: "~{E}"
- board text removed: "~{PHCC}"
- board text removed: "~{PHC}"
- board text removed: "~{PHI}"
- board text removed: "~{PHL}"
- board text removed: "~{PHO}"
- board text removed: "~{PSC}"
- board text removed: "~{PSH}"
- board text removed: "~{PTI}"
- board text removed: "~{PTO}"
- board text removed: "~{SB}"
