File: hardware/interface-board/MEP-MAXI-85V-1-REV-2-Interface-Board.kicad_sch (KiCad schematic)
At the start: 4 parts

Commit message: [feat] Revert to Arduino + add PHY
Removed Arduino Due integration. Added W5500 ENET PHY
Parts:
- renumbered H103 to H102, H102 to H103
Other:
- sheet ATMEL SAM3X8 renamed Arduino Due
- added sheet Interrupt LEDs (interrupt-leds.kicad_sch)
- added sheet WIZnet W5500 ENET PHY (w5500.kicad_sch)
- sheet Arduino Due ports: added 24VRAW, AUX24V, HMI_I2C_SCL1, HMI_I2C_SDA1, HMI_SPI_CS1, HMI_UART_RX1, HMI_UART_RX2, HMI_UART_TX1, HMI_UART_TX2, SPI_MISO, SPI_MOSI, SPI_SCK, ~{12V_ALERT}, ~{3V3_ALERT}, ~{5V_ALERT}, ~{ATSAM3X8E_RESET}, ~{FGND_ALERT}, ~{W5500_INT}, ~{W5500_RST}, ~{W5500_SPI_CS0}; removed ATMEGA16U2-D+, ATMEGA16U2-D-, HMI_RXD, HMI_TXD, MASTER-RESET, MISO, MOSI, SCL1, SDA1, SPCK, SPI1_CS0, VUSBVCC
- sheet External Power ports: added ~{12V_ALERT}, ~{3V3_ALERT}, ~{5V_ALERT}; removed none
- sheet Input Connections ports: added none; removed ESTOP, FUSE
- sheet Output Connections ports: added ESTOP, FUSE, ~{FGND_ALERT}; removed ATMEGA16U2-D+, ATMEGA16U2-D-, FUSED_GND, SBC-USB2-D+, SBC-USB2-D-, VUSB-FUSED
- sheet Pi Zero 2W SBC ports: added 3X8E_I2C_SCL1, 3X8E_I2C_SDA1, 3X8E_SPI_CLK, 3X8E_SPI_CS0, 3X8E_SPI_MISO, 3X8E_SPI_MOSI, 3X8E_UART_RX1, 3X8E_UART_RX2, 3X8E_UART_TX1, 3X8E_UART_TX2; removed Pi-Zero-USB2-D+, Pi-Zero-USB2-D-, SPI1_CLK, SPI1_CS0, SPI1_MISO, SPI1_MOSI, TWI0_SCL/UART2_TX, TWI0_SDA/UART2_RX, UART5_RX, UART5_TX
- sheet Signal Processing ports: added ESTOP*, FUSE*, ~{24VRAW}, ~{AUX24V}; removed none
- note added: "+12V Power Monitor"
- note added: "+3V3V Power Monitor"
- note added: "+5V Power Monitor"
- note added: "07/12/25"
- note added: "12V 5V 3.3V"
- note added: "24VRAW"
- note added: "24VRAW Power Monitor"
- note added: "40h"
- note added: "41h"
- note added: "42h"
- note added: "43h"
- note added: "44h"
- note added: "45h"
- note added: "50h"
- note added: "90h"
- note added: "A401"
- note added: "AT24C256C EEPROM"
- note added: "AUX24V"
- note added: "AUX24V Power Monitor"
- note added: "Address"
- note added: "Arduino Due"
- note added: "Description"
- note added: "Fused GND Power Monitor"
- note added: "I^{2}C Address Muxing"
- note added: "Int"
- note added: "Int/Ext"
- note added: "Ref"
- note added: "Removed Arduino Due integration. Added"
- note added: "U201"
- note added: "U301"
- note added: "U306"
- note added: "U310"
- note added: "U312"
- note added: "U313"
- note added: "U401"
- note added: "W5500 ENET PHY"
- note added: "X3"
- moved on the sheet: H101, H102, H103, H104
