File: hardware/interface-board/arduino_due_io.kicad_sch (KiCad schematic)
At the start: 101 parts, among them IC401 AT24C256C-MAHL-E, J401 TC2030, Q401 DMP3099L, SW401 SW_SPST_Omron_B3FS-100xP, U401 ATmega16U2-M, U402 SN74LVC1G125DCK, U403 SN74LVC1G125DCK, U404 ATSAM3X8EA-AU, Y401 16MHz, Y402 12MHz, Y403 32.768MHz

Commit message: [feat] Revert to Arduino + add PHY
Removed Arduino Due integration. Added W5500 ENET PHY
Parts:
- removed C404, C406, C407, C414, C415, C416, C417, C418, C419, C420, C421, C422, C423, C424, C425, C426, C427, C428, C430, C433, C434, C438: 100nF, Capacitor_SMD:C_0805_2012Metric, symbol Device:C
- removed C405: 1uF, Capacitor_SMD:C_0805_2012Metric, symbol Device:C
- removed C408, C409, C411, C412: 22pF, Capacitor_SMD:C_0805_2012Metric, symbol Device:C
- removed C410: 10pF, Capacitor_SMD:C_0805_2012Metric, symbol Device:C
- removed C413: 10nF, Capacitor_SMD:C_0805_2012Metric, symbol Device:C
- removed C429, C431, C432, C435, C436, C437: 4.7uF, Capacitor_SMD:C_0805_2012Metric, symbol Device:C
- removed D401: 1N4148W, Diode_SMD:D_SOD-323, symbol Device:D
- removed D402: YELLOW, LED_SMD:LED_1206_3216Metric, symbol Device:LED
- removed D403: GREEN, LED_SMD:LED_1206_3216Metric, symbol Device:LED
- removed J401: TC2030, Connector:Tag-Connect_TC2030-IDC-NL_2x03_P1.27mm_Vertical, symbol Connector:TC2030
- removed JP401: Jumper_2_Open, TestPoint:TestPoint_2Pads_Pitch2.54mm_Drill0.8mm, symbol Jumper:Jumper_2_Open
- removed L401, L402, L403: 10uH, Inductor_SMD:L_0805_2012Metric, symbol Device:L
- removed Q401: DMP3099L, Package_TO_SOT_SMD:SOT-23-3, symbol Transistor_FET:DMP3099L
- removed R401, R440: 10K, Resistor_SMD:R_0805_2012Metric, symbol Device:R_US
- removed R402: 1K, Resistor_SMD:R_0805_2012Metric, symbol Device:R_US
- removed R417, R418, R419, R420, R421, R422, R423, R424, R425, R426, R427, R428, R429, R430, R431, R432, R433, R434, R435, R436, R437, R438, R439: 33R, Resistor_SMD:R_0805_2012Metric, symbol Device:R_US
- removed R441, R442, R443: 1R, Resistor_SMD:R_0805_2012Metric, symbol Device:R_US
- removed R444, R445: 4K7, Resistor_SMD:R_0805_2012Metric, symbol Device:R_US
- removed SW401: SW_SPST_Omron_B3FS-100xP, Button_Switch_SMD:SW_SPST_EVQPE1, symbol Switch:SW_Push
- removed U401: ATmega16U2-M, Package_DFN_QFN:QFN-32-1EP_5x5mm_P0.5mm_EP3.6x3.6mm_ThermalVias, symbol MCU_Microchip_ATmega:ATmega16U2-M
- removed U402, U403: SN74LVC1G125DCK, Package_TO_SOT_SMD:Texas_R-PDSO-G5_DCK-5, symbol 74xGxx:SN74LVC1G125DCK
- removed U404: ATSAM3X8EA-AU, ATSAM3X8EA-AU:QFP50P2200X2200X145-144N, symbol ATSAM3X8EA-AU:ATSAM3X8EA-AU
- removed Y401: 16MHz, Crystal:Crystal_SMD_3225-4Pin_3.2x2.5mm, symbol Device:Crystal_GND24
- removed Y402: 12MHz, Crystal:Crystal_SMD_3225-4Pin_3.2x2.5mm, symbol Device:Crystal_GND24
- removed Y403: 32.768MHz, Crystal:Crystal_SMD_3225-4Pin_3.2x2.5mm, symbol Device:Crystal_GND24
- added A401: Arduino_Due_Shield, arduino-library:Arduino_Due_Shield, symbol arduino-library:Arduino_Due_Shield
- added J401: Conn_01x04, Connector_PinSocket_2.54mm:PinSocket_1x04_P2.54mm_Vertical, symbol Connector_Generic:Conn_01x04
- added JP401: SolderJumper_2_Open, Jumper:SolderJumper-2_P1.3mm_Open_TrianglePad1.0x1.5mm, symbol Jumper:SolderJumper_2_Open
- added Q401: SSM6K518NU, SOT-1220UDFN6B_TOS, symbol SSM6K518NU:SSM6K518NU
- added R407, R408: 100R, Resistor_SMD:R_0805_2012Metric, symbol Device:R_US
- added U402, U405, U406, U407, U408, U409, U410, U411, U412, U414: PUSB3BB4Z, PUSB3BB4Z:SON50P100X250X50-10N, symbol PUSB3BB4Z:PUSB3BB4Z
- added U403: APX811-31UG-7, Package_TO_SOT_SMD:SOT-143, symbol APX811-31UG-7:APX811-31UG-7
- added U404: LM74700QDDFRQ1, LM74700QDDFRQ1:SOT65P280X110-8N, symbol LM74700QDDFRQ1:LM74700QDDFRQ1
- C401: value 100nF -> 1uF
- C402: value 22pF -> 0.1uF
- C403: value 22pF -> 100nF; footprint Capacitor_SMD:C_0805_2012Metric -> Capacitor_SMD:C_1206_3216Metric
- R401: renamed from R407; value 4K7 -> 10K
- R402: renamed from R408; value 4K7 -> 10K
- R403: LCSC (none) -> C60816
- R404: value 1K -> 10K; LCSC (none) -> C60816
- R405: value 300R -> 100R
- R406: value 200R -> 100R
- R409: value 6K8 -> 100R
- R410: value 0R -> 100R
- R411: value 100K -> 100R
- R412, R413, R414: value 33R -> 100R
- R415, R416: value 33R -> 10K; LCSC (none) -> C60816
- renumbered IC401 to U401
Connections:
- net D42/PIN42 is gone; now on net SCL: R415.1
- net D43/PIN43 is gone; now on net +3V3: R416.1
- net MASTER-RESET is gone; now on net SCL: R404.2
- net RESET_CMD is gone; now on net +3V3: R404.1
- net USB_BOOT_EN is gone; now on net +3V3: R403.2
- net XTAL1 is gone; now on net GND: C402.1
- net +3V3: now also C401.2, C402.2, R415.2, U403.4 (VCC); no longer R411.2
- net +5V: now also J401.2 (Pin_2); no longer C401.1, R405.2, R406.2
- net AUTO_BUTTON: now also A401.D46
- net ENCODER_BEND_RESET: now also A401.D35, U409.1 (CH1)
- net ENCODER_BEND_SET: now also A401.D34, U408.5 (CH4)
- net ENCODER_FEED_RESET: now also A401.D33, U408.4 (CH3)
- net ENCODER_FEED_SET: now also A401.D32, U408.2 (CH2)
- net ESTOP: now also A401.D47, U411.1 (CH1)
- net FEED_FORWARD: now also R409.2, U406.5 (CH4)
- net FEED_REVERSE: now also R410.2, U407.1 (CH1)
- net FUSE: now also A401.D48, U411.2 (CH2), U411.4 (CH3)
- net GND: now also C401.1, A401.GND1 (GND), A401.GND2 (GND), A401.GND3 (GND), A401.GND4 (SPI_GND), A401.GND5 (GND), A401.GND6 (GND), J401.1 (Pin_1), U402.3 (GND), U402.8 (GND), U403.1 (GND), U404.2 (GND), U405.3 (GND), U405.8 (GND), U406.3 (GND), U406.8 (GND), U407.3 (GND), U407.8 (GND), U408.3 (GND), U408.8 (GND), U409.3 (GND), U409.8 (GND), U410.3 (GND), U410.8 (GND), U411.3 (GND), U411.8 (GND), U412.3 (GND), U412.8 (GND), U414.3 (GND), U414.8 (GND); no longer C401.2, C402.2, C403.2, R403.1, R409.2, R410.2
- net HEAD_CCW: now also R412.2, U407.4 (CH3)
- net HEAD_CW: now also R411.2, U407.2 (CH2)
- net HEAD_IN: now also R414.2, U408.1 (CH1); no longer R412.2
- net HEAD_OUT: now also R413.2, U407.5 (CH4)
- net PROXIMITY_HEAD_CCW: now also A401.D45
- net PROXIMITY_HEAD_CW: now also A401.D44
- net PROXIMITY_HEAD_IN: now also A401.D37, U409.4 (CH3)
- net PROXIMITY_HEAD_LIM: now also A401.D43; no longer R416.2
- net PROXIMITY_HEAD_OUT: now also A401.D36, U409.2 (CH2)
- net PROXIMITY_SHEAR_CUT: now also A401.D39, U410.1 (CH1)
- net PROXIMITY_SHEAR_HOME: now also A401.D38, U409.5 (CH4)
- net PROXIMITY_TOOL_IN: now also A401.D40, U410.2 (CH2)
- net PROXIMITY_TOOL_OUT: now also A401.D41, U410.4 (CH3)
- net SCL: now also A401.D21 (D21/SCL), J401.3 (Pin_3), U414.4 (CH3)
- net SDA: now also R403.1, R416.2, A401.D20 (D20/SDA), J401.4 (Pin_4), U414.5 (CH4)
- net SHEAR_BUTTON: now also A401.D42, U410.5 (CH4); no longer R415.2
- net SHEAR_CUT: now also R405.2, U405.5 (CH4)
- net SHEAR_HOME: now also R406.2, U406.1 (CH1); no longer R413.2
- net TOOL_IN: now also R408.2, U406.4 (CH3)
- net TOOL_OUT: now also R407.2, U406.2 (CH2); no longer R414.2
- net PB26: now reaches R405.1
- net PB26: now also A401.D22
- net PA14: now reaches R406.1
- net PA14: now also A401.D23
- net D23/PIN23 renamed PD9
- net PD9: now also A401.D30
- net D24/PIN24 renamed PA7
- net PA7: now also A401.D31
- net D31/PIN31 renamed PD6
- net PD6: now also A401.D29
- net FWUP renamed PD3
- net PD3: now also A401.D28
- net TST renamed PD2
- net PD2: now also A401.D27
- net VBG renamed PD1
- net PD1: now also A401.D26
- net XTAL2 renamed +12V
- net +12V: now also JP401.1 (A), Q401.1 (D), U404.1 (EN), U404.5 (ANODE)
- new net: C403.2, U404.4 (VCAP)
- new net: Q401.2 (G), U404.6 (GATE)
- new net 24VRAW: A401.D49, U411.5 (CH4)
- new net AUX24V: A401.D50, U412.1 (CH1)
- new net HMI_SPI_CS1: U405.1 (CH1)
- new net PA15: A401.D24, R407.1
- new net PD0: A401.D25, R408.1
- new net SPI_MISO: A401.MISO (SPI_MISO), U402.1 (CH1)
- new net SPI_MOSI: A401.MOSI (SPI_MOSI), U402.2 (CH2)
- new net SPI_SCK: A401.SCK (SPI_SCK), U402.4 (CH3)
- new net VIN: A401.VIN, JP401.2 (B), Q401.3 (S), U404.8 (CATHODE)
- new net X: U412.4 (CH3), U412.5 (CH4)
- new net ~{ATSAM3X8E_RESET}: A401.RST1 (RESET), U403.3 (~{MR}), U412.2 (CH2)
- new net ~{MSD_CS}: A401.D12
- new net ~{MSD_DET}: A401.D13
- new net ~{W5500_INT}: A401.D11, U405.4 (CH3)
- new net ~{W5500_RESET}: U402.5 (CH4)
- new net ~{W5500_RST}: A401.D5, U403.2 (~{RESET})
- new net ~{W5500_SPI_CS0}: A401.D10 (D10_CS0), U405.2 (CH2)
- no-connect marks 24 -> 45
Other:
- note added: "24VRAW"
- note added: "AUX24V"
- note added: "Add a button to reset settings (network)? Add a microSD card slot?"
- note added: "D10/PA28"
- note added: "D11/PD7"
- note added: "D49/PC14"
- note added: "D50/PC13"
- note added: "Remove this?"
- note added: "WIZnet W5500 Reset"
- note added: "~{W5500_INT}"
- note added: "~{W5500_SPI_CS0}"
- note removed: "ATMEGA16U2"
- note removed: "ATMEL SAM3X8"
- note removed: "N.C."
- note removed: "N.C. Internal Pullup"
- moved on the sheet: R401, R402, U401
