File: hardware/interface-board/aux_photoisolators.kicad_sch (KiCad schematic)
At the start: 7 parts, among them IC801 LTV-846S, Q801 BSS138 JI

Commit message: [feat] Revert to Arduino + add PHY
Removed Arduino Due integration. Added W5500 ENET PHY
Parts:
- removed D801: BLUE, LED_SMD:LED_1210_3225Metric, symbol Device:LED
- removed Q801: BSS138 JI, Package_TO_SOT_SMD:SOT-23, symbol Transistor_FET:BSS138
- removed R803: 200R, Resistor_SMD:R_1206_3216Metric, symbol Device:R_US
