File: hardware/interface-board/external_power.kicad_sch (KiCad schematic)
At the start: 35 parts, among them J301 Barrel_Jack_MountingPin, U301 LM1084-ADJ, U302 LM1084-ADJ, U303 LM1084-ADJ

Commit message: [feat] Revert to Arduino + add PHY
Removed Arduino Due integration. Added W5500 ENET PHY
Parts:
- removed C301, C302: 330uF 25V, Capacitor_SMD:CP_Elec_8x10.5, symbol Device:C_Polarized_US
- removed D301, D302, D305: SS10100, Diode_SMD:D_SMC, symbol Device:D_Schottky
- removed D304: SMAZ27-ZJN, Diode_SMD:D_SMA, symbol Device:D_Zener
- removed D307: WHITE, LED_SMD:LED_1210_3225Metric, symbol Device:LED
- removed D309: GREEN, LED_SMD:LED_1210_3225Metric, symbol Device:LED
- removed D311: YELLOW, LED_SMD:LED_1210_3225Metric, symbol Device:LED
- removed L301: 470uH, Inductor_SMD:L_12x12mm_H8mm, symbol Device:L
- removed R304: 200R, Resistor_SMD:R_1206_3216Metric, symbol Device:R_US
- removed R307: 900R, Resistor_SMD:R_1206_3216Metric, symbol Device:R_US
- removed R311: 30R, Resistor_SMD:R_1206_3216Metric, symbol Device:R_US
- added C304, C305, C310, C311: 330uF 25V, Capacitor_SMD:CP_Elec_8x10.5, symbol Device:C_Polarized_US
- added C306, C312, C316: 100nF, Capacitor_SMD:C_1206_3216Metric, symbol Device:C
- added C317, C318: 0.1uF, Capacitor_SMD:C_0805_2012Metric, symbol Device:C
- added C319: 0.012uF, Capacitor_SMD:C_0805_2012Metric, symbol Device:C
- added F301: 16V/1.1A, Fuse:Fuse_1812_4532Metric, symbol Device:Polyfuse
- added J302: Screw_Terminal_01x02, TerminalBlock:TerminalBlock_bornier-2_P5.08mm, symbol Connector:Screw_Terminal_01x02
- added JP301, JP302: SolderJumper_2_Open, Jumper:SolderJumper-2_P1.3mm_Open_TrianglePad1.0x1.5mm, symbol Jumper:SolderJumper_2_Open
- added Q301, Q302: DMT6007LFG, DMT6007LFG:DMP4013LFG7, symbol DMT6007LFG:DMT6007LFG-7
- added Q303: SSM6K518NU, SOT-1220UDFN6B_TOS, symbol SSM6K518NU:SSM6K518NU
- added R303, R308, R314, R327, R328: 2mR, Resistor_SMD:R_2512_6332Metric, symbol Device:R_US
- added R321, R322, R323, R324, R325, R326, R333: 10K, Resistor_SMD:R_0805_2012Metric, symbol Device:R_US
- added R329: 470K, Resistor_SMD:R_0805_2012Metric, symbol Device:R_US
- added R330: 100K, Resistor_SMD:R_0805_2012Metric, symbol Device:R_US
- added R331: 240K, Resistor_SMD:R_0805_2012Metric, symbol Device:R_US
- added R332: 549R, Resistor_SMD:R_0805_2012Metric, symbol Device:R_US
- added R334: 47K, Resistor_SMD:R_0805_2012Metric, symbol Device:R_US
- added R335: 27K, Resistor_SMD:R_0805_2012Metric, symbol Device:R_US
- added U301, U314: INA3221, Package_DFN_QFN:Texas_RGV0016A_VQFN-16-1EP_4x4mm_P0.65mm_EP2.1x2.1mm, symbol Power_Management:INA3221
- added U303, U307, U311: LM74700QDDFRQ1, LM74700QDDFRQ1:SOT65P280X110-8N, symbol LM74700QDDFRQ1:LM74700QDDFRQ1
- added U304, U308: TVS2701DRBR, TVS2701DRBR:IC_TVS2701DRBR, symbol TVS2701DRBR:TVS2701DRBR
- added U312, U313: INA226, Package_SO:VSSOP-10_3x3mm_P0.5mm, symbol Sensor_Energy:INA226
- added U607: LM73100RPWR, LM73100RPWR:IC_LM73100RPWR, symbol LM73100RPWR:LM73100RPWR
- C314: renamed from C308; value 10uF 50V -> 10uF
- D302: renamed from D303; footprint LED_SMD:LED_1210_3225Metric -> LED_SMD:LED_0805_2012Metric
- R307: renamed from R301; footprint Resistor_SMD:R_1206_3216Metric -> Resistor_SMD:R_0805_2012Metric
- renumbered C304 to C302, C307 to C303, C303 to C308, C305 to C309, C306 to C313, D308 to D301, D306 to D303, D310 to D304, R302 to R310, R303 to R311, R308 to R315, R309 to R316, R310 to R318, U301 to U305, U303 to U309
Connections:
- net +12V: now also C316.1, JP301.1 (A), Q303.3 (S), R303.2, U311.1 (EN), U311.5 (ANODE); no longer C303.1, D301.2 (A), R305.1, U302.2 (VO)
- net +24V: now also D302.2 (A), C304.1, C310.1, Q301.3 (D), Q302.3 (D), U303.8 (CATHODE), U307.8 (CATHODE)
- net +3V3: now also C317.2, C318.2, R314.2, R321.2, R322.1, R323.1, R324.2, R325.1, R326.1, R333.1, U312.2 (A0), U312.6 (VS), U313.6 (VS); no longer C314.1, D304.2 (A), R315.1, U309.2 (VO)
- net +5V: now also R308.2; no longer C309.1, D303.2 (A), R310.1, U305.2 (VO)
- net 24VRAW: now also R328.1, U304.1 (IN), U304.2 (IN), U304.3 (IN), U304.4 (IN), U313.10 (Vin+), U313.8 (Vbus)
- net GND: now also J301.3 (MountPin), C304.2, C305.2, C310.2, C311.2, C317.1, C318.1, C319.2, J302.2 (Pin_2), R331.2, R332.2, R335.2, U303.2 (GND), U304.5 (GND), U304.6 (GND), U304.7 (GND), U304.8 (GND), U307.2 (GND), U308.5 (GND), U308.6 (GND), U308.7 (GND), U308.8 (GND), U311.2 (GND), U312.1 (A1), U312.7 (GND), U313.1 (A1), U313.2 (A0), U313.7 (GND), U607.8 (GND); no longer J301.MP (MountPin)
- net AUX24V: now reaches J301.1
- net AUX24V: now also R327.1, U308.1 (IN), U308.2 (IN), U308.3 (IN), U308.4 (IN), U312.10 (Vin+), U312.8 (Vbus)
- new net: C306.2, U303.4 (VCAP)
- new net: R330.2, R331.1, U607.2 (OVLO)
- new net: R329.2, R330.1, U607.1 (EN/UVLO)
- new net: R334.2, R335.1, U607.4 (PGTH)
- new net: C316.2, U311.4 (VCAP)
- new net: Q303.2 (G), U311.6 (GATE)
- new net: Q301.2 (G), U303.6 (GATE)
- new net: C319.1, U607.7 (DVDT)
- new net: Q302.2 (G), U307.6 (GATE)
- new net: C312.2, U307.4 (VCAP)
- new net +12V-HMI-FUSED: F301.2, J302.1 (Pin_1)
- new net 12V: F301.1, JP301.2 (B), Q303.1 (D), U311.8 (CATHODE)
- new net 12VOUT: C303.1, D301.2 (A), R303.1, R305.1, U302.2 (VO)
- new net 24VRAWSHUNT: C305.1, C306.1, Q301.1 (S), R328.2, U303.1 (EN), U303.5 (ANODE), U313.9 (Vin-)
- new net 3V3IMON: R332.1, U607.9 (IMON)
- new net 3V3OUT: JP302.2 (B), R314.1, R334.1, U607.6 (OUT)
- new net 3V3OUTPG: R333.2, U607.3 (PG)
- new net 3V3VO: C314.1, D304.2 (A), JP302.1 (A), R315.1, R329.1, U309.2 (VO), U607.5 (IN)
- new net 5VOUT: C309.1, D303.2 (A), R308.1, R310.1, U305.2 (VO)
- new net AUX24VSHUNT: C311.1, C312.1, Q302.1 (S), R327.2, U307.1 (EN), U307.5 (ANODE), U312.9 (Vin-)
- new net SCL: R322.2, R325.2, U312.5 (SCL), U313.5 (SCL)
- new net SDA: R321.1, R324.1, U312.4 (SDA), U313.4 (SDA)
- new net ~{24VRAW_ALERT}: R326.2, U313.3 (~{Alert})
- new net ~{AUX24V_ALERT}: R323.2, U312.3 (~{Alert})
Other:
- note added: "+12V Rail"
- note added: "+3V3 Rail"
- note added: "+5V Rail"
- note added: "24V ORing"
- note added: "24VRAW Power & Current Monitor"
- note added: "300R: RT1206BRD07300RL 2K580: RN73H2BTTD2581F100 Use 0.1% resistors"
- note added: "300R: RT1206BRD07300RL 470R: RT1206BRD07470RL 22R: CPF1206B22RE1 Use 0.1% resistors"
- note added: "300R: RT1206BRD07300RL 900R: PAT1206E9000BST1 Use 0.1% resistors"
- note added: "AUX24V Power & Current Monitor"
- note added: "Addr: 1000000b (40h)"
- note added: "Addr: 1000001b (41h)"
- note added: "HMI Screen"
- note added: "R_{1}"
- note added: "R_{2}"
- note added: "R_{3}"
- note added: "R_{4}"
- note added: "R_{5}"
- note added: "R_{IMON}(Ω) = (1.5V x 10^{-6}) / (5A x 182) = 549R"
- note added: "Where V_{PGTH(R)} = 1.2V, R_{4} = 47K 3.3 = 1.2V x (47000 + R_{5}) / R_{5} R_{5} = 26,857 R_{5} = 27K"
- note added: "Where V_{UVLO(R)} = 1.2V V_{OV(R)} = 1.2V R_{1} = 470K R_{2} = 100K UV: 3V = 1.2V x (470000 + 100000 + R_{3}) / (100000 + R_{3}) R_{2} = 213,333 OV: 4V = 1.2V x (470000 + 100000 + R_{3}) / (R_{3}) R_{3} = 244,286 So, R_{3} = 240K"
- note added: "Where t_{r} (ms) = 20 mS SR = 3.3 V / 20 mS = 0.165 V/mS C_{dVdt}(pF) = 2000 / SR (V/mS) = 2000 / 0.165 = 12,121pF / 0.012uF"
- note removed: "12V Rail"
- note removed: "24V Rail"
- note removed: "3V3 Rail"
- note removed: "5V Rail"
- note removed: "LEDS: 2-3V @20mA Half Brightness: 3V3 @ 10mA = 30R Half Brightness: 5V @ 10mA = 200R Half Brightness: 12V @ 10mA = 900R Half Brightness: 24V @ 10mA = 2100R"
- note removed: "Notes"
- note removed: "R301: RT1206BRD07300RL R302: PAT1206E9000BST1"
- note removed: "R303: RT1206BRD07300RL R304: RN73H2BTTD2581F100"
- note removed: "R305: RT1206BRD07300RL R306: RT1206BRD07470RL R307: CPF1206B22RE1"
- note removed: "Supposed to be 2K1"
- note removed: "Use 0.1% resistors"
- moved on the sheet: C302, C303, C308, C309, C313, C314, D301, D302, D303, D304, J301, R305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
