File: hardware/interface-board/input_connections.kicad_sch (KiCad schematic)
At the start: 3 parts, among them J501 Conn_02x10_Odd_Even, J502 Screw_Terminal_01x02

Commit message: [feat] Revert to Arduino + add PHY
Removed Arduino Due integration. Added W5500 ENET PHY
Parts:
- removed F501: 3512P, Fuse:Fuseholder_Clip-5x20mm_Keystone_3512P_Inline_P23.62x7.27mm_D1.02x2.41x1.02x1.57mm_Horizontal, symbol Device:Fuse
- removed J502: Screw_Terminal_01x02, TerminalBlock:TerminalBlock_bornier-2_P5.08mm, symbol Connector:Screw_Terminal_01x02
- added U501, U502, U503, U504: PUSB3BB4Z, PUSB3BB4Z:SON50P100X250X50-10N, symbol PUSB3BB4Z:PUSB3BB4Z
Connections:
- net AUTO_BUTTON: now also U502.5 (CH4)
- net ENCODER_BEND_RESET: now also U503.2 (CH2)
- net ENCODER_BEND_SET: now also U501.2 (CH2)
- net ENCODER_FEED_RESET: now also U503.1 (CH1)
- net ENCODER_FEED_SET: now also U501.1 (CH1)
- net GND: now also U501.3 (GND), U501.8 (GND), U502.3 (GND), U502.8 (GND), U503.3 (GND), U503.8 (GND), U504.3 (GND), U504.8 (GND)
- net PROXIMITY_HEAD_CCW: now also U504.4 (CH3)
- net PROXIMITY_HEAD_CW: now also U502.4 (CH3)
- net PROXIMITY_HEAD_IN: now also U503.4 (CH3)
- net PROXIMITY_HEAD_LIM: now also U504.2 (CH2)
- net PROXIMITY_HEAD_OUT: now also U501.4 (CH3)
- net PROXIMITY_SHEAR_CUT: now also U503.5 (CH4)
- net PROXIMITY_SHEAR_HOME: now also U501.5 (CH4)
- net PROXIMITY_TOOL_IN: now also U502.1 (CH1)
- net PROXIMITY_TOOL_OUT: now also U504.1 (CH1)
- net SHEAR_BUTTON: now also U502.2 (CH2)
- new net: U501.10, U503.10
- new net: U501.6, U503.6
- new net: U501.7, U503.7
- new net: U501.9, U503.9
- new net: U502.10, U504.10
- new net: U502.6, U504.6
- new net: U502.7, U504.7
- new net: U502.9, U504.9
- no-connect marks 2 -> 3
Other:
- note added: "ESD PROTECTION"
- note removed: "ESTOP"
- note removed: "ESTOP to be wired for NC"
- moved on the sheet: J501
