File: hardware/interface-board/output_connections.kicad_sch (KiCad schematic)
At the start: 60 parts, among them J201 USB_C_Receptacle_USB2.0_16P, J202 Conn_02x07_Odd_Even, J203 Screw_Terminal_01x02, Q201 IRFR7540TRPBF, Q202 IRFR7540TRPBF, Q203 IRFR7540TRPBF, Q204 IRFR7540TRPBF, Q205 IRFR7540TRPBF, Q206 IRFR7540TRPBF, Q207 IRFR7540TRPBF, Q208 IRFR7540TRPBF, Q209 IRFR7540TRPBF, Q210 IRFR7540TRPBF, U201 USBLC6-2SC6

Commit message: [feat] Revert to Arduino + add PHY
Removed Arduino Due integration. Added W5500 ENET PHY
Parts:
- removed J201: USB_C_Receptacle_USB2.0_16P, Connector_USB:USB_C_Receptacle_G-Switch_GT-USB-7010ASV, symbol Connector:USB_C_Receptacle_USB2.0_16P
- removed J203: Screw_Terminal_01x02, TerminalBlock:TerminalBlock_bornier-2_P5.08mm, symbol Connector:Screw_Terminal_01x02
- removed JP201, JP202: Jumper_3_Open, Connector_PinHeader_2.54mm:PinHeader_1x03_P2.54mm_Vertical, symbol Jumper:Jumper_3_Open
- removed L201: 470uH, Inductor_SMD:L_12x12mm_H8mm, symbol Device:L
- removed R222: 5K1, Resistor_SMD:R_0805_2012Metric, symbol Device:R_US
- removed U201: USBLC6-2SC6, Package_TO_SOT_SMD:SOT-23-6, symbol Power_Protection:USBLC6-2SC6
- added C201: 0.1uF, Capacitor_SMD:C_0805_2012Metric, symbol Device:C
- added J202: Screw_Terminal_01x02, TerminalBlock:TerminalBlock_bornier-2_P5.08mm, symbol Connector:Screw_Terminal_01x02
- added R219, R224: 10K, Resistor_SMD:R_0805_2012Metric, symbol Device:R_US
- added R220: 2mR, Resistor_SMD:R_2512_6332Metric, symbol Device:R_US
- added U201: INA226, Package_SO:VSSOP-10_3x3mm_P0.5mm, symbol Sensor_Energy:INA226
- added U202, U203, U204, U205: PUSB3BB4Z, PUSB3BB4Z:SON50P100X250X50-10N, symbol PUSB3BB4Z:PUSB3BB4Z
- D201: footprint LED_SMD:LED_1210_3225Metric -> LED_SMD:LED_0805_2012Metric
- D202: renamed from D209; footprint LED_SMD:LED_1210_3225Metric -> LED_SMD:LED_0805_2012Metric
- D203: renamed from D217; footprint LED_SMD:LED_1210_3225Metric -> LED_SMD:LED_0805_2012Metric
- D207: renamed from D203; footprint LED_SMD:LED_1210_3225Metric -> LED_SMD:LED_0805_2012Metric
- D208: renamed from D211; footprint LED_SMD:LED_1210_3225Metric -> LED_SMD:LED_0805_2012Metric
- D209: renamed from D219; footprint LED_SMD:LED_1210_3225Metric -> LED_SMD:LED_0805_2012Metric
- D213: renamed from D205; footprint LED_SMD:LED_1210_3225Metric -> LED_SMD:LED_0805_2012Metric
- D214: renamed from D213; footprint LED_SMD:LED_1210_3225Metric -> LED_SMD:LED_0805_2012Metric
- D217: renamed from D207; footprint LED_SMD:LED_1210_3225Metric -> LED_SMD:LED_0805_2012Metric
- D218: renamed from D215; footprint LED_SMD:LED_1210_3225Metric -> LED_SMD:LED_0805_2012Metric
- F201: value 500mA -> 3512P; footprint Fuse:Fuse_1812_4532Metric -> Fuse:Fuseholder_Clip-5x20mm_Keystone_3512P_Inline_P23.62x7.27mm_D1.02x2.41x1.02x1.57mm_Horizontal
- R201: renamed from R205; footprint Resistor_SMD:R_1206_3216Metric -> Resistor_SMD:R_0805_2012Metric
- R202: renamed from R213; footprint Resistor_SMD:R_1206_3216Metric -> Resistor_SMD:R_0805_2012Metric
- R203: renamed from R219; footprint Resistor_SMD:R_1206_3216Metric -> Resistor_SMD:R_0805_2012Metric
- R204: renamed from R201; footprint Resistor_SMD:R_1206_3216Metric -> Resistor_SMD:R_0805_2012Metric
- R205: renamed from R209; footprint Resistor_SMD:R_1206_3216Metric -> Resistor_SMD:R_0805_2012Metric
- R206: renamed from R217; footprint Resistor_SMD:R_1206_3216Metric -> Resistor_SMD:R_0805_2012Metric
- R207: renamed from R206; footprint Resistor_SMD:R_1206_3216Metric -> Resistor_SMD:R_0805_2012Metric
- R208: renamed from R214; footprint Resistor_SMD:R_1206_3216Metric -> Resistor_SMD:R_0805_2012Metric
- R209: renamed from R220; footprint Resistor_SMD:R_1206_3216Metric -> Resistor_SMD:R_0805_2012Metric
- R210: renamed from R202; footprint Resistor_SMD:R_1206_3216Metric -> Resistor_SMD:R_0805_2012Metric
- R211: renamed from R210; footprint Resistor_SMD:R_1206_3216Metric -> Resistor_SMD:R_0805_2012Metric
- R212: renamed from R218; footprint Resistor_SMD:R_1206_3216Metric -> Resistor_SMD:R_0805_2012Metric
- R213: renamed from R207; footprint Resistor_SMD:R_1206_3216Metric -> Resistor_SMD:R_0805_2012Metric
- R214: renamed from R215; footprint Resistor_SMD:R_1206_3216Metric -> Resistor_SMD:R_0805_2012Metric
- R215: renamed from R203; footprint Resistor_SMD:R_1206_3216Metric -> Resistor_SMD:R_0805_2012Metric
- R216: renamed from R211; footprint Resistor_SMD:R_1206_3216Metric -> Resistor_SMD:R_0805_2012Metric
- R217: renamed from R208; footprint Resistor_SMD:R_1206_3216Metric -> Resistor_SMD:R_0805_2012Metric
- R218: renamed from R216; footprint Resistor_SMD:R_1206_3216Metric -> Resistor_SMD:R_0805_2012Metric
- R221: value 5K1 -> 10K; LCSC (none) -> C1489
- R222: renamed from R204; footprint Resistor_SMD:R_1206_3216Metric -> Resistor_SMD:R_0805_2012Metric
- R223: renamed from R212; footprint Resistor_SMD:R_1206_3216Metric -> Resistor_SMD:R_0805_2012Metric
- renumbered D202 to D204, D210 to D205, D218 to D206, D204 to D210, D212 to D211, D220 to D212, D206 to D215, D214 to D216, D208 to D219, D216 to D220, J202 to J201, Q205 to Q202, Q209 to Q203, Q202 to Q204, Q206 to Q205, Q210 to Q206, Q203 to Q207, Q207 to Q208, Q204 to Q209, Q208 to Q210
Connections:
- net +5V: no longer R203.1, R209.1
- net FUSED_GND: now also R220.1, U201.10 (Vin+)
- net GND: now also R203.2, R209.2, C201.1, J202.1 (Pin_1), U201.7 (GND), U202.3 (GND), U202.8 (GND), U203.3 (GND), U203.8 (GND), U204.3 (GND), U204.8 (GND), U205.3 (GND), U205.8 (GND); no longer R221.1
- net HEAD_IN: now also D209.2 (A)
- net HEAD_OUT: now also D203.2 (A)
- net SOL_FEED_FORWARD: now also U202.4 (CH3)
- net SOL_FEED_REVERSE: now also U203.4 (CH3)
- net SOL_HEAD_CCW: now also U203.5 (CH4)
- net SOL_HEAD_CW: now also U202.5 (CH4)
- net SOL_HEAD_IN: now also U204.2 (CH2); no longer D209.1 (K)
- net SOL_HEAD_OUT: now also U204.1 (CH1); no longer D203.1 (K)
- net SOL_SHEER_CUT: now also U202.1 (CH1)
- net SOL_SHEER_HOME: now also U203.1 (CH1)
- net SOL_TOOL_IN: now also U203.2 (CH2)
- net SOL_TOOL_OUT: now also U202.2 (CH2)
- net SCL: now reaches R221.2
- net SCL: now also U201.5 (SCL)
- net VUSB renamed FUSE
- net FUSE: now also R220.2, U201.9 (Vin-)
- net VUSB-FUSED renamed ESTOP
- net ESTOP: now also J202.2 (Pin_2), U205.1 (CH1)
- new net: D203.1 (K), R203.1
- new net: D209.1 (K), R209.1
- new net +24V: U201.8 (Vbus)
- new net +3V3: C201.2, R219.2, R221.1, R224.1, U201.1 (A1), U201.2 (A0), U201.6 (VS)
- new net SDA: R219.1, U201.4 (SDA)
- new net ~{FGND_ALERT}: R224.2, U201.3 (~{Alert})
- no-connect marks 3 -> 6
Other:
- note added: "Addr: 1000101b (45h)"
- note added: "ESTOP"
- note added: "ESTOP to be wired for NC"
- note added: "Optional ESD protection"
- note added: "Power & Current Monitor"
- note removed: "ATMEGA16U2 USBC & SELECTOR"
- note removed: "HMI Screen"
- moved on the sheet: D201, D202, D203, D204, D205, D206, D207, D208, D209, D210, D211, D212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
