File: hardware/interface-board/photoisolators.kicad_sch (KiCad schematic)
At the start: 93 parts, among them IC701 LTV-846S, IC702 LTV-846S, IC703 LTV-846S, IC704 LTV-846S, IC801 LTV-846S, Q701 BSS138 JI, Q702 BSS138 JI, Q703 BSS138 JI, Q704 BSS138 JI, Q705 BSS138 JI, Q706 BSS138 JI, Q707 BSS138 JI, Q708 BSS138 JI, Q709 BSS138 JI, Q710 BSS138 JI, Q711 BSS138 JI, Q712 BSS138 JI, Q713 BSS138 JI, Q714 BSS138 JI, Q715 BSS138 JI, Q716 BSS138 JI, Q801 BSS138 JI

Commit message: [feat] Revert to Arduino + add PHY
Removed Arduino Due integration. Added W5500 ENET PHY
Parts:
- removed D701, D702, D703, D704, D705, D706, D707, D708, D709, D710, D711, D712, D713, D714, D715, D716, D801: BLUE, LED_SMD:LED_1210_3225Metric, symbol Device:LED
- removed IC701, IC702, IC703, IC704, IC801: LTV-846S, LTV-846S:LTV846S, symbol LTV-846S:LTV-846S
- removed Q701, Q702, Q703, Q704, Q705, Q706, Q707, Q708, Q709, Q710, Q711, Q712, Q713, Q714, Q715, Q716, Q801: BSS138 JI, Package_TO_SOT_SMD:SOT-23, symbol Transistor_FET:BSS138
- removed R701, R702, R711, R712, R713, R714, R715, R716, R717, R718, R719, R720, R729, R730, R731, R732, R803: 200R, Resistor_SMD:R_1206_3216Metric, symbol Device:R_US
- removed R703, R704, R705, R706, R707, R708, R709, R710, R721, R722, R723, R724, R725, R726, R727, R728, R801: 1K2, Resistor_SMD:R_0805_2012Metric, symbol Device:R_US
Connections:
- no-connect marks 12 -> 0
Other:
- note removed: "1K140: RN73R2ATTD1141D25"
- note removed: "Interrupt LED Indicators"
- note removed: "Interrupt LEDS: 2-3V @20mA Half Brightness: 3V @ 10mA = 200R 75% Brightness: 3V @ 15mA = 133.3R"
- note removed: "LTV-846S +V Value: 24V LED Voltage Drop: 1.2V LED Current: 20mA Resistor Value: 1K140 Alternative Value: 1K2"
- note removed: "Notes"
