File: hardware/interface-board/pi-zero-w2.kicad_sch (KiCad schematic)
At the start: 34 parts, among them J601 USB_C_Receptacle_USB2.0_16P, J602 RJ45_Amphenol_RJMG1BD3B8K1ANR, J603 Conn_02x05_Odd_Even, J604 Conn_Coaxial, J605 Conn_01x24_MountingPin, Q601 BSS138 JI, SW601 SW_SPST_Omron_B3FS-100xP, U601 USBLC6-2SC6, U602 CH340E, U603 RASPBERRY_PI_ZERO_2_W

Commit message: [feat] Revert to Arduino + add PHY
Removed Arduino Due integration. Added W5500 ENET PHY
Parts:
- removed C601: 10uF, Capacitor_Tantalum_SMD:CP_EIA-3216-10_Kemet-I, symbol Device:C_Polarized_US
- removed C604, C605: 0.1uF, Capacitor_SMD:C_0805_2012Metric, symbol Device:C
- removed C608, C609: 470uF, Capacitor_SMD:CP_Elec_4x5.4, symbol Device:C_Polarized
- removed D601: GREEN, LED_SMD:LED_1206_3216Metric, symbol Device:LED
- removed D602: SS34, Diode_SMD:D_SMA, symbol Device:D_Schottky
- removed F601: 500mA, Fuse:Fuse_1812_4532Metric, symbol Device:Fuse
- removed J601: USB_C_Receptacle_USB2.0_16P, Connector_USB:USB_C_Receptacle_G-Switch_GT-USB-7010ASV, symbol Connector:USB_C_Receptacle_USB2.0_16P
- removed J602: RJ45_Amphenol_RJMG1BD3B8K1ANR, Connector_RJ:RJ45_Amphenol_RJMG1BD3B8K1ANR, symbol Connector:RJ45_Amphenol_RJMG1BD3B8K1ANR
- removed JP601: Jumper_2_Bridged, TestPoint:TestPoint_2Pads_Pitch2.54mm_Drill0.8mm, symbol Jumper:Jumper_2_Bridged
- removed L601: 470uH, Inductor_SMD:L_12x12mm_H8mm, symbol Device:L
- removed R601: 0, Resistor_SMD:R_0805_2012Metric, symbol Device:R_US
- removed R602: 30R, Resistor_SMD:R_0805_2012Metric, symbol Device:R_US
- removed R603, R604: 5K1, Resistor_SMD:R_0805_2012Metric, symbol Device:R_US
- removed R609: 4K7, Resistor_SMD:R_0805_2012Metric, symbol Device:R_US
- removed U601: USBLC6-2SC6, Package_TO_SOT_SMD:SOT-23-6, symbol Power_Protection:USBLC6-2SC6
- removed U602: CH340E, Package_SO:MSOP-10_3x3mm_P0.5mm, symbol Interface_USB:CH340E
- added C601: 100nF, Capacitor_SMD:C_1206_3216Metric, symbol Device:C
- added C603: 100nF, Capacitor_SMD:C_0805_2012Metric, symbol Device:C
- added FB601: 330R, Inductor_SMD:L_0805_2012Metric, symbol Device:FerriteBead
- added J604: USB_A, Connector_USB:USB_A_Connfly_DS1095, symbol Connector:USB_A
- added J605: RJ45_Hanrun_HR911105A_Horizontal, Connector_RJ:RJ45_Hanrun_HR911105A_Horizontal, symbol Connector:RJ45_Hanrun_HR911105A_Horizontal
- added JP601: SolderJumper_2_Open, Jumper:SolderJumper-2_P1.3mm_Open_TrianglePad1.0x1.5mm, symbol Jumper:SolderJumper_2_Open
- added Q601: SSM6K518NU, SOT-1220UDFN6B_TOS, symbol SSM6K518NU:SSM6K518NU
- added R607: 10K, Resistor_SMD:R_0805_2012Metric, symbol Device:R_US
- added U601: LM74700QDDFRQ1, LM74700QDDFRQ1:SOT65P280X110-8N, symbol LM74700QDDFRQ1:LM74700QDDFRQ1
- added U603, U606: USBLC6-2SC6, Package_TO_SOT_SMD:SOT-23-6, symbol Power_Protection:USBLC6-2SC6
- added U604: MIC2005A-1YM5-TR, SOT95P280X145-5N, symbol MIC2005A-1YM5-TR:MIC2005A-1YM5-TR
- added U605: PUSB3BB4Z, PUSB3BB4Z:SON50P100X250X50-10N, symbol PUSB3BB4Z:PUSB3BB4Z
- R608: value 4K7 -> 10K; LCSC C60816 -> (none)
- renumbered C603 to C604, C607 to C605, J605 to J601, J604 to J602, Q601 to Q602, R605 to R603, R610 to R604, R606 to R605, R607 to R606, U603 to U602
Connections:
- net VUSB-FUSED is gone; now on net GND: C606.1
- net +3V3: now also R608.1, R607.1; no longer R608.2
- net +5V: now also C601.1, JP601.1 (A), Q601.1 (D), U601.1 (EN), U601.5 (ANODE); no longer J603.8 (Pin_8)
- net D+: now also J604.3 (D+), U603.1 (I/O1)
- net D-: now also J604.2 (D-), U603.3 (I/O2)
- net EPHY-RXN: now also J605.6 (RD-)
- net EPHY-RXP: now also J605.3 (RD+)
- net EPHY-TXN: now also J605.2 (TD-)
- net EPHY-TXP: now also J605.1 (TD+)
- net GND: now also C603.1, J604.4 (GND), J604.5 (Shield), J605.10, J605.11, J605.8, J605.SH, U601.2 (GND), U603.2 (GND), U604.2 (GND), U605.3 (GND), U605.8 (GND), U606.2 (GND); no longer C606.2
- net PWRSW: now also U605.4 (CH3)
- net TWI2_SCL/UART3_TX: now also U605.2 (CH2)
- net TWI2_SDA/UART3_RX: now also U605.1 (CH1)
- net USB3-D+: now also U606.6 (I/O1); no longer J603.4 (Pin_4)
- net USB3-D-: now also U606.4 (I/O2); no longer J603.3 (Pin_3)
- net at R605.1: now also J605.9
- net at C604.1: now also J605.5 (RCT)
- net 5V: now reaches U602.2 (5V_2), U602.4 (5V_4)
- net 5V: now also C606.2, J603.8 (Pin_8), JP601.2 (B), Q601.3 (S), U601.8 (CATHODE), U604.1 (VIN), U606.5 (VBUS)
- net at C602.1: now also J605.4 (TCT)
- net at R603.1: now also J605.12
- net PI13 renamed ~{USB_FAULT}
- net ~{USB_FAULT}: now also R607.2, U604.6 (~{FAULT})
- net PI15 renamed USB_EN
- net USB_EN: now also R608.2, U604.3 (EN)
- net PWM1: no longer names the net of U602.32 (GPIO12)
- net Pi-Zero-USB2-D+ renamed USB2-D+
- net USB2-D+: now also U603.6 (I/O1)
- net Pi-Zero-USB2-D- renamed USB2-D-
- net USB2-D-: now also U603.4 (I/O2)
- net SCL renamed TWI1_SCL
- net SDA renamed TWI1_SDA
- net TWI1_SDA: no longer R608.1
- net SPI1_CLK: no longer names the net of U602.23 (GPIO11/SPI_SCLK)
- net SPI1_CS0: no longer names the net of U602.24 (GPIO8/SPI_~{CE0})
- net SPI1_MISO: no longer names the net of U602.21 (GPIO9/SPI_MISO)
- net SPI1_MOSI: no longer names the net of U602.19 (GPIO10/SPI_MOSI)
- net TWI0_SCL/UART2_TX: no longer names the net of U602.15 (GPIO22/GPIO_GEN3)
- net TWI0_SDA/UART2_RX: no longer names the net of U602.22 (GPIO25/GPIO_GEN6)
- net UART5_RX: no longer names the net of U602.13 (GPIO27/GPIO_GEN2)
- net UART5_TX: no longer names the net of U602.11 (GPIO17/GPIO_GEN0)
- new net: C601.2, U601.4 (VCAP)
- new net: C603.2, FB601.1, J604.1 (VBUS), U603.5 (VBUS)
- new net: Q601.2 (G), U601.6 (GATE)
- new net: FB601.2, U604.5 (VOUT)
- new net USB-D+: J603.4 (Pin_4), U606.1 (I/O1)
- new net USB-D-: J603.3 (Pin_3), U606.3 (I/O2)
- no-connect marks 7 -> 6
Other:
- note added: "Ideal Diode"
- note added: "TWI0_SCL/UART2_TX"
- note added: "TWI0_SDA/UART2_RX"
- note added: "TWI1_SCL"
- note added: "TWI1_SDA"
- note added: "UART5_RX"
- note added: "UART5_TX"
- note added: "USB 2.0 Type-A Connector"
- note removed: "Debug UART Console"
- note removed: "To ATSAM3X8E"
- moved on the sheet: C602, C604, C605, J601, J602, J603, Q602, R603, R604, R605, R606, SW601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
