File: hardware/interface-board/signal-processing.kicad_sch (KiCad schematic)
At the start: 170 parts, among them IC701 LTV-846S, IC702 LTV-846S, IC703 LTV-846S, IC704 LTV-846S, IC705 LTV-846S, Q701 BSS138 JI, Q702 BSS138 JI, Q703 BSS138 JI, Q704 BSS138 JI, Q705 BSS138 JI, Q706 BSS138 JI, Q707 BSS138 JI, Q708 BSS138 JI, Q709 BSS138 JI, Q710 BSS138 JI, Q711 BSS138 JI, Q712 BSS138 JI, Q713 BSS138 JI, Q714 BSS138 JI, Q715 BSS138 JI, Q716 BSS138 JI, Q717 BSS138 JI, U701 SN74HC14PWR, U702 SN74HC14PWR, U703 SN74HC14PWR

Commit message: [feat] Revert to Arduino + add PHY
Removed Arduino Due integration. Added W5500 ENET PHY
Parts:
- removed C717, C720, C721, C722: 47uF, Capacitor_SMD:C_0805_2012Metric, symbol Device:C
- removed D701, D702, D703, D704, D705, D706, D707, D708, D709, D710, D711, D712, D713, D714, D715, D716: BLUE, LED_SMD:LED_1210_3225Metric, symbol Device:LED
- removed D717: RED, LED_SMD:LED_1210_3225Metric, symbol Device:LED
- removed Q701, Q702, Q703, Q704, Q705, Q706, Q707, Q708, Q709, Q710, Q711, Q712, Q713, Q714, Q715, Q716, Q717: BSS138 JI, Package_TO_SOT_SMD:SOT-23, symbol Transistor_FET:BSS138
- removed R705, R706, R707, R708, R710, R711, R715, R716, R717: 1K2, Resistor_SMD:R_0805_2012Metric, symbol Device:R_US
- removed R718, R721, R722, R740, R741, R744, R745, R746, R747, R748, R749, R750, R751: 200R, Resistor_SMD:R_1206_3216Metric, symbol Device:R_US
- removed TP701, TP702, TP703, TP704, TP705, TP717, TP718, TP719, TP720, TP730, TP731, TP732, TP733, TP743, TP744, TP745, TP746: Orange, TestPoint:TestPoint_THTPad_D1.0mm_Drill0.5mm, symbol Connector:TestPoint
- removed TP706, TP707, TP708, TP709, TP710, TP721, TP722, TP723, TP724, TP734, TP735, TP736, TP737, TP747, TP748, TP749, TP750: Yellow, TestPoint:TestPoint_THTPad_D1.0mm_Drill0.5mm, symbol Connector:TestPoint
- removed TP711, TP712, TP713, TP714, TP715, TP725, TP726, TP727, TP728, TP738, TP739, TP740, TP741, TP751, TP752, TP753, TP754: White, TestPoint:TestPoint_THTPad_D1.0mm_Drill0.5mm, symbol Connector:TestPoint
- removed TP716, TP729: Red, TestPoint:TestPoint_THTPad_D3.0mm_Drill1.5mm, symbol Connector:TestPoint
- removed TP742, TP755: Black, TestPoint:TestPoint_THTPad_D3.0mm_Drill1.5mm, symbol Connector:TestPoint
- added C716: 1uF, Capacitor_SMD:C_0805_2012Metric, symbol Device:C
- added R723, R724, R725, R730, R731, R736: 105R, Resistor_SMD:R_0805_2012Metric, symbol Device:R_US
- added R733: 100K, Resistor_SMD:R_0805_2012Metric, symbol Device:R_US
- added R737, R738: 1K2, Resistor_SMD:R_1206_3216Metric, symbol Device:R_US
- added U708: 74LVC1G14GW-Q100,1, Package_TO_SOT_SMD:SOT-353_SC-70-5, symbol 74xGxx:74AHC1G14
- C701: renamed from C714; value 47uF -> 1uF
- C704: renamed from C715; value 47uF -> 1uF
- C711: renamed from C716; value 47uF -> 1uF
- C718, C719: value 47uF -> 1uF
- R701, R702, R703, R709, R712, R713, R714: value 1K2 -> 105R
- R708: renamed from R704; value 1K2 -> 105R
- R719, R735: value 200R -> 105R; footprint Resistor_SMD:R_1206_3216Metric -> Resistor_SMD:R_0805_2012Metric; LCSC C844654 -> (none)
- R720: value 200R -> 105R; footprint Resistor_SMD:R_1206_3216Metric -> Resistor_SMD:R_0805_2012Metric
- R734: value 200R -> 100K; footprint Resistor_SMD:R_1206_3216Metric -> Resistor_SMD:R_0805_2012Metric; LCSC C844654 -> (none)
- renumbered C701 to C702, C706 to C703, C702 to C705, C707 to C706, C711 to C707, C713 to C708, C703 to C709, C708 to C710, C704 to C712, C709 to C713, C710 to C714, C712 to C715, C705 to C717, R723 to R704, R730 to R705, R736 to R706, R742 to R707, R724 to R710, R729 to R711, R725 to R715, R731 to R716, R738 to R717, R743 to R718, R726 to R721, R732 to R722, R727 to R726, R733 to R727, R737 to R728, R739 to R729, R728 to R732, IC701 to U701, U701 to U702, IC702 to U703, U702 to U704, IC703 to U705, U703 to U706, IC704 to U707, IC705 to U709
Connections:
- net +24V is gone; now on net +3V3: R701.1, R702.1, R703.1, R708.1, R709.1, R712.1, R713.1, R714.1
- net +3V3: now also R719.1, R720.1, R734.1, R735.1, C716.1, R723.1, R724.1, R725.1, R730.1, R731.1, R733.1, R736.1, U708.5 (VCC); no longer C718.2, C719.2
- net 24VRAW: now also R737.1
- net GND: now also C718.2, C719.2, U709.11 (E3), U709.13 (E2), U709.4 (C2), U709.6 (C3), C716.2, U708.3 (GND); no longer C718.1, C719.1, U706.13 (6A)
- net at U705.3 (A2): now also R720.2
- net ~{24VRAW}: now reaches U706.12 (6Y)
- net at U705.5 (A3): now also R723.2
- net at U707.5 (A3): now also R731.2
- net at R714.2: now also U703.7 (A4); no longer U707.3 (A_2)
- net at U705.1 (A1): now also R719.2; no longer R709.2
- net at U707.7 (A4): now also R735.2
- net at U709.1 (A1): now also R736.2
- net AUX24V*: now reaches U709.12 (C3)
- net AUX24V*: now also C719.1, R734.2, U708.2
- net 24VRAW*: now reaches U709.14 (C2)
- net 24VRAW*: now also C718.1, U706.13 (6A), R733.2
- net at U709.3 (A2): now also R737.2
- net at U709.5 (A3): now also R738.2
- net at R712.2: now also U703.3 (A2); no longer U705.7 (A_4)
- net at U703.1 (A1): now also R709.2
- net at U703.5 (A3): now also R713.2
- net at U707.1 (A1): now also R725.2; no longer R713.2
- removed net +5V: R719.2, R720.2, R734.2, R735.2
- new net: R730.2, U707.3 (A2)
- new net: R724.2, U705.7 (A4)
- new net AUX24V: R738.1
- new net ~{AUX24V}: U708.4
- no-connect marks 13 -> 4
Other:
- note added: "LTV-846S +V Value: 3.3V LED Voltage Drop: 1.2V LED Current: 20mA Resistor Value: 105R Alternative Value: 110R"
- note removed: "1K140: RN73R2ATTD1141D25"
- note removed: "Interrupt LED Indicators"
- note removed: "Interrupt LEDS: 2-3V @20mA Half Brightness: 3V @ 10mA = 200R 75% Brightness: 3V @ 15mA = 133.3R"
- note removed: "LTV-846S +V Value: 24V LED Voltage Drop: 1.2V LED Current: 20mA Resistor Value: 1K140 Alternative Value: 1K2"
- note removed: "Notes"
- note removed: "Test Points"
- moved on the sheet: C701, C702, C703, C704, C705, C706, C707, C708, C709, C710, C711, C712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
