File: hardware/keypad/debounce.kicad_sch (KiCad schematic)
At the start: 108 parts, among them SW401 DISPLAY, SW402 RUN, SW403 LEFT, SW404 MEMORY, SW405 COMP, SW406 UP, SW407 MENU, SW408 DOWN, SW409 INFEED, SW410 ENTER, SW411 RIGHT, SW412 DECIMAL, SW413 HEAD_POS, SW414 1, SW415 4, SW416 7, SW417 FTI, SW418 2, SW419 5, SW420 8, SW421 SHEAR, SW422 3, SW423 6, SW424 9, SW425 PAUSE, SW426 PLUS, SW427 MINUS, SW428 0, U401 SN74HC14PWR, U402 SN74HC14PWR, U403 SN74HC14PWR, U404 SN74HC14PWR, U405 SN74HC14PWR, U406 SN74LVC2G14DBV, U407 PCF8575DBR, U408 PCF8575DBR, U409 74LVC1G32GW,125

Commit message: Revision X2!
New and improved revision of the keypad! I fixed issues with the repeater and remote SBC power switch circuit (hopefully🤞). I also integrated the Arduino Nano onto the board (ATMEGA328).
Connections:
- net ~{INT1}: now also U406.6 (1Y), U409.1; no longer R430.2, U406.1 (1A), U408.1 (~{INT})
- net ~{INT2}: now also U406.4 (2Y), U409.2; no longer R429.2, U406.3 (2A), U407.1 (~{INT})
- net INT renamed PCF8575_INT
- new net INT1: R430.2, U406.1 (1A), U408.1 (~{INT})
- new net INT2: R429.2, U406.3 (2A), U407.1 (~{INT})
Other:
- moved on the sheet: C401, C402, C403, C404, C405, C406, C407, C408, C409, C410, C411, C412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
