File: hardware/keypad/keypad.kicad_pcb (KiCad board)
At the start: 4 copper layers, 209 x 97.3 mm, 167 parts, among them J101 Conn_02x05_Odd_Even, Q301 BSS83P, Q302 BSS83P, Q501 BSS83P, Q502 BSS138 JI, SW401 DISPLAY, SW402 RUN, SW403 LEFT, SW404 MEMORY, SW405 COMP, SW406 UP, SW407 MENU, SW408 DOWN, SW409 INFEED, SW410 ENTER, SW411 RIGHT, SW412 DECIMAL, SW413 HEAD_POS, SW414 1, SW415 4, SW416 7, SW417 FTI, SW418 2, SW419 5, SW420 8, SW421 SHEAR, SW422 3, SW423 6, SW424 9, SW425 PAUSE, SW426 PLUS, SW427 MINUS, SW428 0, U301 SN74HCS4075DR, U302 SN74HCS4075DR, U303 SN74HCS4075DR, U304 SN74LVC2G14DBV, U305 LMC555xM, U306 SN74LVC2G14DBVR, U401 SN74HC14PWR, U402 SN74HC14PWR, U403 SN74HC14PWR, U404 SN74HC14PWR, U405 SN74HC14PWR, U406 SN74LVC2G14DBV, U407 PCF8575DBR, U408 PCF8575DBR, U409 74LVC1G32GW,125, U501 NL17SZ08, U502 SN74LVC2G14DBV, U503 LMC555xM

Commit message: Revision X2!
New and improved revision of the keypad! I fixed issues with the repeater and remote SBC power switch circuit (hopefully🤞). I also integrated the Arduino Nano onto the board (ATMEGA328).
Parts:
- removed A101: Arduino_Nano_v3.x, Module:Arduino_Nano
- removed C101, C102, C103, C104, C105, C106, C502: 1uF, Capacitor_SMD:C_0805_2012Metric
- removed Q301, Q302, Q501: BSS83P, Package_TO_SOT_SMD:SOT-23
- removed R501: 10K, Resistor_SMD:R_0805_2012Metric
- removed TP102: Red, TestPoint:TestPoint_Keystone_5000-5004_Miniature
- removed TP506: Yellow, TestPoint:TestPoint_Keystone_5000-5004_Miniature
- removed U502: SN74LVC2G14DBV, SN74LVC2G14DBVR:SOT95P280X145-6N
- added C201: 100nF, Capacitor_SMD:C_0805_2012Metric, F.Cu at (68.6, 81.6)
- added C202: 4.7uF, Capacitor_SMD:C_0805_2012Metric, F.Cu at (68.6, 83.6)
- added C203: 100nF, Capacitor_SMD:C_0805_2012Metric, F.Cu at (52.4, 74.1)
- added C204: 100nF, Capacitor_SMD:C_0805_2012Metric, F.Cu at (70.2, 97.2)
- added C205: 100nF, Capacitor_SMD:C_0805_2012Metric, F.Cu at (72.2, 97.2)
- added C309: 100nF, Capacitor_SMD:C_0805_2012Metric, F.Cu at (72.5, 60.4)
- added C310: 1uF, Capacitor_SMD:C_0805_2012Metric, F.Cu at (63.0, 123.8)
- added C311: 0.1uF, Capacitor_SMD:C_0805_2012Metric, F.Cu at (56.4, 128.3)
- added C601: 100nF, Capacitor_SMD:C_0805_2012Metric, F.Cu at (68.2, 97.2)
- added C602: 22pF, Capacitor_SMD:C_0805_2012Metric, F.Cu at (54.6, 95.2)
- added C603: 22pF, Capacitor_SMD:C_0805_2012Metric, F.Cu at (50.4, 98.5)
- added D101: SR240 SS24, Diode_SMD:D_SMA, F.Cu at (78.4, 56.4)
- added D201: RED, LED_SMD:LED_0805_2012Metric, F.Cu at (72.2, 76.0)
- added D202: GREEN, LED_SMD:LED_0805_2012Metric, F.Cu at (72.2, 78.2)
- added D602: Orange, LED_SMD:LED_0805_2012Metric, F.Cu at (58.5, 104.6)
- added F301: 500mA, Fuse:Fuse_0805_2012Metric, F.Cu at (56.8, 63.9)
- added J201: TC2030, Connector:Tag-Connect_TC2030-IDC-NL_2x03_P1.27mm_Vertical, F.Cu at (69.9, 104.4)
- added J301: USB_C_Receptacle_USB2.0_16P, Connector_USB:USB_C_Receptacle_G-Switch_GT-USB-7010ASV, F.Cu at (48.2, 65.9)
- added L301: 10uH, Inductor_SMD:L_0805_2012Metric, F.Cu at (60.7, 63.9)
- added R101: 10K, Resistor_SMD:R_0805_2012Metric, F.Cu at (77.5, 47.0)
- added R102: 10K, Resistor_SMD:R_0805_2012Metric, F.Cu at (81.9, 47.0)
- added R103: 0R, Resistor_SMD:R_0805_2012Metric, F.Cu at (81.2, 56.4)
- added R201: 130R, Resistor_SMD:R_0805_2012Metric, F.Cu at (68.6, 76.0)
- added R202: 30R, Resistor_SMD:R_0805_2012Metric, F.Cu at (68.6, 78.2)
- added R306: 1M, Resistor_SMD:R_0805_2012Metric, F.Cu at (54.4, 128.3)
- added R602: 130R, Resistor_SMD:R_0805_2012Metric, F.Cu at (61.2, 103.8)
- added R604: 10K, Resistor_SMD:R_0805_2012Metric, F.Cu at (62.4, 88.9)
- added R609: 250R, Resistor_SMD:R_0805_2012Metric, F.Cu at (63.2, 103.8)
- added R610: 250R, Resistor_SMD:R_0805_2012Metric, F.Cu at (65.2, 103.8)
- added R611: 250R, Resistor_SMD:R_0805_2012Metric, F.Cu at (69.0, 100.2)
- added R612: 250R, Resistor_SMD:R_0805_2012Metric, F.Cu at (60.4, 88.9)
- added R613: 250R, Resistor_SMD:R_0805_2012Metric, F.Cu at (58.4, 88.9)
- added R614: 250R, Resistor_SMD:R_0805_2012Metric, F.Cu at (56.4, 88.9)
- added R615: 250R, Resistor_SMD:R_0805_2012Metric, F.Cu at (53.9, 91.8)
- added TP308: 125-00868, TestPoint:TestPoint_Keystone_5000-5004_Miniature, F.Cu at (73.4, 64.1)
- added U201: FT232RL, Package_SO:SSOP-28_5.3x10.2mm_P0.65mm, F.Cu at (60.4, 77.7)
- added U307: AMS1117-3.3, Package_TO_SOT_SMD:SOT-223-3_TabPin2, F.Cu at (67.0, 62.3)
- added U308: NC7SZ00M5X, Package_TO_SOT_SMD:SOT-23-5, F.Cu at (59.7, 126.1)
- added U601: ATMEGA328-AU, Package_QFP:TQFP-32_7x7mm_P0.8mm, F.Cu at (61.8, 96.6)
- added Y601: 20MHz, Crystal:Crystal_SMD_3225-4Pin_3.2x2.5mm, F.Cu at (53.6, 98.7)
- C304, C308: value 1uF -> 100nF
- C307: value .47uF -> 1uF
- C503: footprint Capacitor_SMD:C_0805_2012Metric -> Capacitor_SMD:C_Elec_6.3x5.4
- D501: value LED -> RED
- R301, R302: value 10K -> 5K1
- R304: value 330K -> 10K
- R305: value 10K -> 22K
- TP305: value Yellow -> 125-00869
- TP306: value White -> 125-00868
- U304: value SN74LVC2G14DBV -> NC7SZ00M5X; footprint SN74LVC2G14DBVR:SOT95P280X145-6N -> Package_TO_SOT_SMD:SOT-23-5
- U305, U503: value LMC555xM -> LMC555CMX/NOPB
- U306: value SN74LVC2G14DBVR -> USBLC6-2SC6; footprint SN74LVC2G14DBVR:SOT95P280X145-6N -> Package_TO_SOT_SMD:SOT-23-6; moved to B.Cu
- U501: value NL17SZ08 -> NC7SZ08M5X
- moved R301 66.1 mm to (49.0, 57.6), turned to 0 degrees
- moved R302 60.9 mm to (49.0, 59.6), turned to 0 degrees
- moved TP306 57.3 mm to (68.2, 68.1)
- moved TP305 56.4 mm to (58.4, 58.3)
- moved U306 53.3 mm to (58.9, 66.9)
- moved C304 52.9 mm to (60.0, 69.7)
- moved C308 49.6 mm to (63.8, 67.8), turned to -90 degrees
- moved R502 38.6 mm to (81.0, 120.2), turned to -90 degrees
- moved C504 35.6 mm to (81.0, 116.6), turned to -90 degrees
- moved R504 34.9 mm to (81.6, 124.1), turned to -90 degrees
- moved D501 34.4 mm to (80.2, 128.0), turned to 180 degrees
- moved Q502 32.9 mm to (78.5, 123.4)
- moved R503 32.9 mm to (75.4, 123.4)
- moved TP504 32.0 mm to (72.6, 122.2)
- moved U503 31.7 mm to (76.0, 117.4)
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Connections:
- net Net-(U305-THR) renamed /Repeater/THRESHOLD_~{TRIGGER}
- net Net-(U503-THR) renamed /Pi Zero 2W Power Reset/THRESHOLD_~{TRIGGER}
- C304 pad 1: +5V -> GND
- C304 pad 2: GND -> Net-(U306-VBUS)
- C307 pad 1: Net-(U306-1A) -> +5V
- J101 pad 7: /TWI2_SDA -> SDA
- J101 pad 8: +5V -> Net-(D101-A)
- J101 pad 9: /TWI2_SCL -> SCL
- R301 pad 1: /Repeater/DELAY -> GND
- R301 pad 2: GND -> Net-(J301-CC1)
- R302 pad 1: +5V -> GND
- R302 pad 2: Net-(Q301-G) -> Net-(J301-CC2)
- R304 pad 1: /REPEAT_INT -> /Repeater/GATE
- R304 pad 2: Net-(U306-1A) -> GND
- R305 pad 1: /Repeater/GOSC_VCC -> Net-(R305-Pad1)
- R305 pad 2: +5V -> Net-(C311-Pad2)
- R429 pad 2: /Debounce Switches/~{INT2} -> /Debounce Switches/INT2
- R430 pad 2: /Debounce Switches/~{INT1} -> /Debounce Switches/INT1
- TP301 pad 1: Net-(U303-3Y) -> /Repeater/3Y_RESET
- TP302 pad 1: /Repeater/DELAY -> /Repeater/3Y_RESET
- TP303 pad 1: /Repeater/GOSC_VCC -> /Repeater/GATE
- TP305 pad 1: Net-(Q301-G) -> GND
- TP306 pad 1: Net-(Q302-D) -> +5V
- TP307 pad 1: /REPEAT_INT -> /REPEATER_INT
- TP503 pad 1: Net-(U502-1A) -> /Pi Zero 2W Power Reset/~{MEMORY}&~{DOWN}
- U303 pad 10: Net-(U303-3Y) -> /Repeater/3Y_RESET
- U304 pad 1: Net-(U303-3Y) -> /Repeater/GATE
- U304 pad 2: GND -> Net-(R305-Pad1)
- U304 pad 3: /Repeater/DELAY -> GND
- U304 pad 4: /Repeater/GOSC_VCC -> Net-(R306-Pad1)
- U305 pad 3: /Repeater/DELAY -> /Repeater/GATE
- U305 pad 4: +5V -> /Repeater/3Y_RESET
- U305 pad 8: Net-(Q301-D) -> +5V
- U306 pad 1: Net-(U306-1A) -> /USB3-D+
- U306 pad 3: GND -> /USB3-D-
- U306 pad 4: unconnected-(U306-2Y-Pad4) -> /Microcontroller/D-
- U306 pad 5: Net-(Q302-D) -> Net-(U306-VBUS)
- U306 pad 6: /REPEAT_INT -> /Microcontroller/D+
- U406 pad 1: /Debounce Switches/~{INT1} -> /Debounce Switches/INT1
- U406 pad 3: /Debounce Switches/~{INT2} -> /Debounce Switches/INT2
- U406 pad 4: Net-(U406-2Y) -> /Debounce Switches/~{INT2}
- U406 pad 6: Net-(U406-1Y) -> /Debounce Switches/~{INT1}
- U407 pad 1: /Debounce Switches/~{INT2} -> /Debounce Switches/INT2
- U408 pad 1: /Debounce Switches/~{INT1} -> /Debounce Switches/INT1
- U409 pad 1: Net-(U406-1Y) -> /Debounce Switches/~{INT1}
- U409 pad 2: Net-(U406-2Y) -> /Debounce Switches/~{INT2}
- U409 pad 4: /INT -> /PCF8575_INT
- U501 pad 4: Net-(U502-1A) -> /Pi Zero 2W Power Reset/~{MEMORY}&~{DOWN}
- U503 pad 4: +5V -> /Pi Zero 2W Power Reset/~{MEMORY}&~{DOWN}
- U503 pad 8: Net-(Q501-D) -> +5V
Routing:
- net /Repeater/3Y_RESET: track 0.00 -> 310.3 mm, vias 0 -> 2
- net Net-(U303-3Y): track 307.9 -> 0.00 mm, vias 2 -> 0
- net /PCF8575_INT: track 0.00 -> 78.3 mm, vias 0 -> 3
- net /INT: track 75.4 -> 0.00 mm, vias 1 -> 0
- net /REPEATER_INT: track 0.00 -> 66.6 mm
- net /Microcontroller/~{RESET}/PC6: track 0.00 -> 61.9 mm, vias 0 -> 5
- net /USB3-D-: track 0.00 -> 44.4 mm, vias 0 -> 1
- net /USB3-D+: track 0.00 -> 44.4 mm, vias 0 -> 1
- net /REPEAT_INT: track 43.6 -> 0.00 mm, vias 1 -> 0
- net /Debounce Switches/INT1: track 0.00 -> 38.1 mm, vias 0 -> 2
- net /Repeater/DELAY: track 36.3 -> 0.00 mm
- net /Debounce Switches/~{INT1}: track 38.1 -> 1.85 mm, vias 2 -> 0
- net /PWRSW: track 44.7 -> 80.8 mm, vias 2 -> 3
- net +5V: track 68.6 -> 96.0 mm
- net /Debounce Switches/INT2: track 0.00 -> 27.0 mm, vias 0 -> 2
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- added copper zone on F.Cu, net +3V3
- added copper zone on F.Cu, net +5V
Other:
- board text added: "HEARTBEAT"
- board text added: "Keypad Hardware & Firmware: Connor McMillan Rev X2"
- board text added: "RX"
- board text added: "SBC PWRSW"
- board text added: "TX"
- board text removed: "Keypad Hardware & Firmware: Connor McMillan Rev X1"
