File: hardware/keypad/keypad.kicad_pcb (KiCad board)
At the start: 4 copper layers, 209 x 97.3 mm, 192 parts, among them J101 Conn_02x05_Odd_Even, J201 TC2030, J301 USB_C_Receptacle_USB2.0_16P, Q502 BSS138 JI, SW401 DISPLAY, SW402 RUN, SW403 LEFT, SW404 MEMORY, SW405 COMP, SW406 UP, SW407 MENU, SW408 DOWN, SW409 INFEED, SW410 ENTER, SW411 RIGHT, SW412 DECIMAL, SW413 HEAD_POS, SW414 1, SW415 4, SW416 7, SW417 FTI, SW418 2, SW419 5, SW420 8, SW421 SHEAR, SW422 3, SW423 6, SW424 9, SW425 PAUSE, SW426 PLUS, SW427 MINUS, SW428 0, U201 FT232RL, U301 SN74HCS4075DR, U302 SN74HCS4075DR, U303 SN74HCS4075DR, U304 NC7SZ00M5X, U305 LMC555CMX/NOPB, U306 USBLC6-2SC6, U307 AMS1117-3.3, U308 NC7SZ00M5X, U401 SN74HC14PWR, U402 SN74HC14PWR, U403 SN74HC14PWR, U404 SN74HC14PWR, U405 SN74HC14PWR, U406 SN74LVC2G14DBV, U407 PCF8575DBR, U408 PCF8575DBR, U409 74LVC1G32GW,125, U501 NC7SZ08M5X, U503 LMC555CMX/NOPB, U601 ATMEGA328-AU, Y601 20MHz

Commit message: [fix] repeater and sbc shutdown circuit
Fixed repeater and SBC shutdown circuit. Switched +5V VCC to +3.3V. Added C211
Parts:
- removed the C308 at (63.8, 67.8)
- removed D101: SR240 SS24, Diode_SMD:D_SMA
- removed L301: 10uH, Inductor_SMD:L_0805_2012Metric
- removed R103: 0R, Resistor_SMD:R_0805_2012Metric
- removed the TP302 at (59.6, 112.7)
- removed TP308: 125-00868, TestPoint:TestPoint_Keystone_5000-5004_Miniature
- added C101: 22uF, Capacitor_SMD:C_1206_3216Metric, F.Cu at (79.1, 68.2)
- added C102: 22uF, Capacitor_SMD:C_1206_3216Metric, B.Cu at (77.9, 57.1)
- added C103: 100nF, Capacitor_SMD:C_1206_3216Metric, F.Cu at (77.9, 57.1)
- added C201: 22uF, Capacitor_SMD:C_1206_3216Metric, F.Cu at (63.8, 68.4)
- added C203: 22uF, Capacitor_SMD:C_1206_3216Metric, B.Cu at (52.6, 58.2)
- added C204: 100nF, Capacitor_SMD:C_1206_3216Metric, F.Cu at (52.6, 58.2)
- added C211: 100nF, Capacitor_SMD:C_0805_2012Metric, F.Cu at (66.2, 82.1)
- added C301: 1uF, Capacitor_SMD:C_0805_2012Metric, F.Cu at (46.0, 118.5)
- added C501: 1uF, Capacitor_SMD:C_0805_2012Metric, F.Cu at (78.0, 112.0)
- added FB201: 330R, Inductor_SMD:L_0805_2012Metric, F.Cu at (57.4, 62.8)
- added JP101: SolderJumper_2_Open, Jumper:SolderJumper-2_P1.3mm_Open_TrianglePad1.0x1.5mm, F.Cu at (81.2, 60.7)
- added JP201: SolderJumper_2_Open, Jumper:SolderJumper-2_P1.3mm_Open_TrianglePad1.0x1.5mm, F.Cu at (55.6, 55.2)
- added Q101: DMT6007LFG, DMT6007LFG:DMP4013LFG7, F.Cu at (77.6, 64.7)
- added Q201: DMT6007LFG, DMT6007LFG:DMP4013LFG7, F.Cu at (60.2, 58.6)
- added Q301: PMV30XPEAR, Package_TO_SOT_SMD:SOT-23-3, F.Cu at (49.7, 121.0)
- added Q501: PMV30XPEAR, Package_TO_SOT_SMD:SOT-23-3, F.Cu at (81.8, 114.3)
- added U101: LM74700QDDFRQ1, LM74700QDDFRQ1:SOT65P280X110-8N, F.Cu at (78.0, 60.5)
- added U202: LM74700QDDFRQ1, LM74700QDDFRQ1:SOT65P280X110-8N, F.Cu at (55.9, 58.2)
- added U301: 74LVC1G14GW-Q100,1, Package_TO_SOT_SMD:SOT-353_SC-70-5, F.Cu at (46.0, 121.0)
- added U501: 74LVC1G14GW-Q100,1, Package_TO_SOT_SMD:SOT-353_SC-70-5, F.Cu at (78.1, 114.4)
- R204: renamed from R609; value 250R -> 270R
- R205: renamed from R610; value 250R -> 270R
- R206: renamed from R611; value 250R -> 270R
- R208: renamed from R612; value 250R -> 270R
- R209: renamed from R613; value 250R -> 270R
- R210: renamed from R614; value 250R -> 270R
- R211: renamed from R615; value 250R -> 270R
- R501: renamed from R504; value 150R -> 130
- Y201: renamed from Y601; value 20MHz -> 16MHz
- moved TP202 41.8 mm to (84.2, 91.2)
- moved TP505 36.7 mm to (55.3, 137.4)
- moved C214 17.9 mm to (52.4, 76.1), turned to 180 degrees
- moved C213 16.6 mm to (52.4, 78.1), turned to 180 degrees
- moved TP304 14.4 mm to (51.1, 133.1)
- moved R304 13.1 mm to (61.1, 121.2), turned to 0 degrees
- moved C307 12.0 mm to (60.4, 118.4), turned to -90 degrees
- moved C309 8.32 mm to (64.7, 128.9)
- moved TP504 4.53 mm to (67.8, 114.3)
- moved TP503 4.18 mm to (82.0, 108.8)
- moved C306 3.40 mm to (61.2, 124.7), turned to 0 degrees
- moved TP302 3.32 mm to (50.4, 126.7)
- moved R303 2.90 mm to (57.1, 129.4), turned to 180 degrees
- moved C504 2.66 mm to (69.0, 119.8)
- moved U305 2.62 mm to (57.3, 126.7)
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- renumbered C309 to C202, C304 to C205, C601 to C206, C204 to C207, C205 to C208, C602 to C209, C603 to C210, C203 to C212, C201 to C213, C202 to C214, C301 to C302, C310 to C304, C306 to C305, C307 to C306, C305 to C307, C302 to C308, C311 to C309, C429 to C401, C436 to C402, C430 to C403, C401 to C404, C409 to C406, C413 to C407, C417 to C408, C421 to C409, C425 to C410, C434 to C411, C437 to C412, C414 to C413, C402 to C414, C406 to C415, C410 to C416, C418 to C417, C422 to C418, C426 to C419, C431 to C420, C403 to C421, C407 to C422, C411 to C423, C415 to C424, C419 to C425, C423 to C426, C432 to C428, C404 to C429, C408 to C430, C412 to C431, C416 to C432, C420 to C433, C424 to C434, C428 to C435, C435 to C436, C433 to C437, C504 to C502, C501 to C503, C503 to C504, D602 to D201, D201 to D202, D202 to D203, F301 to F201, J301 to J201, J201 to J202, R301 to R201, R302 to R202, R602 to R203, R604 to R207, R201 to R212, R202 to R213, R304 to R301, R305 to R302, R306 to R303, R303 to R304, R430 to R401, R433 to R402, R434 to R403, R401 to R404, R409 to R406, R413 to R407, R417 to R408, R421 to R409, R425 to R410, R414 to R411, R402 to R412, R406 to R413, R410 to R414, R418 to R415, R422 to R416, R426 to R417, R403 to R418, R407 to R419, R411 to R420, R415 to R421, R419 to R422, R427 to R424, R429 to R425, R404 to R426, R408 to R427, R412 to R428, R416 to R429, R420 to R430, R424 to R431, R428 to R432, R431 to R433, R432 to R434, R503 to R502, R502 to R503, SW405 to SW402, SW409 to SW403, SW413 to SW404, SW417 to SW405, SW421 to SW406, SW425 to SW407, SW414 to SW408, SW402 to SW409, SW406 to SW410, SW410 to SW411, SW418 to SW412, SW422 to SW413, SW426 to SW414, SW403 to SW415, SW407 to SW416, SW411 to SW417, SW415 to SW418, SW423 to SW420, SW427 to SW421, SW404 to SW422, SW408 to SW423, SW412 to SW424, SW416 to SW425, SW420 to SW426, SW424 to SW427, TP103 to TP102, TP306 to TP201, TP305 to TP202, TP303 to TP302, TP304 to TP303, TP307 to TP304, TP504 to TP501, TP501 to TP502, TP502 to TP504, U307 to U201, U306 to U203, U601 to U204, U201 to U205, U301 to U302, U308 to U303, U303 to U304, U304 to U305, U305 to U306, U302 to U307, U408 to U402, U402 to U403, U406 to U404, U409 to U405, U403 to U406, U404 to U408, U405 to U409, U501 to U502
Connections:
- net /Repeater/GATE renamed /Repeater/OSC_GATE
- net Net-(F301-Pad1) renamed /Microcontroller/VBUS
- net Net-(J301-CC1) renamed /Microcontroller/CC1
- net Net-(J301-CC2) renamed /Microcontroller/CC2
- net Net-(U306-VBUS) renamed /Microcontroller/FVBUS
- C206 pad 1: +5V -> +3V3
- C207 pad 1: +5V -> +3V3
- C208 pad 1: +5V -> +3V3
- C213 pad 1: +5V -> +3V3
- C214 pad 1: +5V -> +3V3
- C302 pad 2: +5V -> +3V3
- C303 pad 2: +5V -> +3V3
- C304 pad 1: +5V -> +3V3
- C305 pad 1: +5V -> /Repeater/GATED_VCC
- C306 pad 1: +5V -> +3V3
- C307 pad 1: +5V -> /Repeater/GATED_VCC
- C308 pad 2: +5V -> +3V3
- C401 pad 1: +5V -> +3V3
- C402 pad 2: +5V -> +3V3
- C403 pad 1: +5V -> +3V3
- C411 pad 2: +5V -> +3V3
- C412 pad 2: +5V -> +3V3
- C420 pad 1: +5V -> +3V3
- C428 pad 1: +5V -> +3V3
- C436 pad 2: +5V -> +3V3
- C437 pad 1: +5V -> +3V3
- C502 pad 1: +5V -> /Pi Zero 2W Power Reset/GATED_VCC
- C503 pad 1: +5V -> +3V3
- C504 pad 1: +5V -> /Pi Zero 2W Power Reset/GATED_VCC
- D501 pad 2: +5V -> +3V3
- J101 pad 8: Net-(D101-A) -> /5VCC
- J202 pad 2: +5V -> +3V3
- R101 pad 1: +5V -> +3V3
- R102 pad 2: +5V -> +3V3
- R207 pad 1: +5V -> +3V3
- R401 pad 1: +5V -> +3V3
- R402 pad 1: +5V -> +3V3
- R403 pad 2: +5V -> +3V3
- R404 pad 1: +5V -> +3V3
- R405 pad 1: +5V -> +3V3
- R406 pad 1: +5V -> +3V3
- R407 pad 1: +5V -> +3V3
- R408 pad 1: +5V -> +3V3
- R409 pad 1: +5V -> +3V3
- R410 pad 1: +5V -> +3V3
- R411 pad 1: +5V -> +3V3
- R412 pad 1: +5V -> +3V3
- R413 pad 1: +5V -> +3V3
- R414 pad 1: +5V -> +3V3
- R415 pad 1: +5V -> +3V3
- R416 pad 1: +5V -> +3V3
- R417 pad 1: +5V -> +3V3
- R418 pad 1: +5V -> +3V3
- R419 pad 1: +5V -> +3V3
- R420 pad 1: +5V -> +3V3
- R421 pad 1: +5V -> +3V3
- R422 pad 1: +5V -> +3V3
- R423 pad 1: +5V -> +3V3
- R424 pad 1: +5V -> +3V3
- R425 pad 1: +5V -> +3V3
- R426 pad 1: +5V -> +3V3
- R427 pad 1: +5V -> +3V3
- R428 pad 1: +5V -> +3V3
- R429 pad 1: +5V -> +3V3
- R430 pad 1: +5V -> +3V3
- R431 pad 1: +5V -> +3V3
- R432 pad 1: +5V -> +3V3
- R433 pad 1: +5V -> +3V3
- R434 pad 2: +5V -> +3V3
- TP101 pad 1: +5V -> +3V3
- U204 pad 18: +5V -> +3V3
- U204 pad 4: +5V -> +3V3
- U204 pad 6: +5V -> +3V3
- U205 pad 15: /Microcontroller/D- -> /Microcontroller/D+
- U205 pad 16: /Microcontroller/D+ -> /Microcontroller/D-
- U205 pad 17: unconnected-(U201-3V3OUT-Pad17) -> +3V3
- U205 pad 24: (no net) -> unconnected-(U205-Pad24)
- U205 pad 4: +5V -> +3V3
- U205 pad 8: (no net) -> unconnected-(U205-Pad8)
- U302 pad 14: +5V -> +3V3
- U303 pad 5: +5V -> +3V3
- U304 pad 14: +5V -> +3V3
- U305 pad 5: +5V -> +3V3
- U306 pad 4: /Repeater/3Y_RESET -> /Repeater/GATED_VCC
- U306 pad 8: +5V -> /Repeater/GATED_VCC
- U307 pad 14: +5V -> +3V3
- U401 pad 14: +5V -> +3V3
- U402 pad 24: +5V -> +3V3
- U403 pad 14: +5V -> +3V3
- U404 pad 5: +5V -> +3V3
- U405 pad 5: +5V -> +3V3
- U406 pad 14: +5V -> +3V3
- U407 pad 21: +5V -> +3V3
- U407 pad 24: +5V -> +3V3
- U408 pad 14: +5V -> +3V3
- U409 pad 11: +5V -> +3V3
- U409 pad 13: +5V -> +3V3
- U409 pad 14: +5V -> +3V3
- U502 pad 5: +5V -> +3V3
- U503 pad 4: /Pi Zero 2W Power Reset/~{MEMORY}&~{DOWN} -> /Pi Zero 2W Power Reset/GATED_VCC
- U503 pad 8: +5V -> /Pi Zero 2W Power Reset/GATED_VCC
Routing:
- net +5V: track 96.0 -> 23.6 mm, vias 64 -> 0
- net +3V3: track 20.4 -> 87.5 mm, vias 0 -> 64
- net /Repeater/3Y_RESET: track 310.3 -> 250.6 mm, vias 2 -> 1
- net /Pi Zero 2W Power Reset/GATED_VCC: track 0.00 -> 26.2 mm, vias 0 -> 2
- net /Repeater/GATED_VCC: track 0.00 -> 21.3 mm
- net /5VCC: track 0.00 -> 13.7 mm, vias 0 -> 1
- net Net-(C309-Pad2): track 4.02 -> 13.0 mm, vias 0 -> 2
- net /Pi Zero 2W Power Reset/THRESHOLD_~{TRIGGER}: track 12.4 -> 19.5 mm
- net /Microcontroller/FBFVBUS: track 0.00 -> 6.22 mm, vias 0 -> 1
- net /REPEATER_INT: track 66.6 -> 60.6 mm, vias 0 -> 1
- net Net-(D101-A): track 5.99 -> 0.00 mm
- net /Repeater/GATE: track 0.00 -> 5.10 mm
- net /Pi Zero 2W Power Reset/GATE: track 0.00 -> 4.78 mm
- net /Microcontroller/D+: track 25.4 -> 29.9 mm
- net /Microcontroller/D-: track 25.4 -> 29.9 mm
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- added copper zone on In2.Cu, net +3V3
- added copper zone on F.Cu, net /5VCC
- added copper zone on F.Cu, net /Microcontroller/FBFVBUS
- added copper zone on F.Cu, net /Microcontroller/FVBUS
- added copper zone on F.Cu, net /Microcontroller/VBUS
- removed copper zone on In2.Cu, net +5V
Other:
- board text added: "Keypad Rev X3 MADE IN U.S.A"
- board text removed: "Keypad Hardware & Firmware: Connor McMillan Rev X2"
