File: hardware/keypad/microcontroller.kicad_sch (KiCad schematic)
At the start: 39 parts, among them J201 TC2030, J301 USB_C_Receptacle_USB2.0_16P, U201 FT232RL, U306 USBLC6-2SC6, U307 AMS1117-3.3, U601 ATMEGA328-AU, Y601 20MHz

Commit message: [fix] repeater and sbc shutdown circuit
Fixed repeater and SBC shutdown circuit. Switched +5V VCC to +3.3V. Added C211
Parts:
- removed C308: 100nF, Capacitor_SMD:C_0805_2012Metric, symbol Device:C
- removed L301: 10uH, Inductor_SMD:L_0805_2012Metric, symbol Device:L
- removed TP308: 125-00868, TestPoint:TestPoint_Keystone_5000-5004_Miniature, symbol Connector:TestPoint
- added C201, C203: 22uF, Capacitor_SMD:C_1206_3216Metric, symbol Device:C
- added C204: 100nF, Capacitor_SMD:C_1206_3216Metric, symbol Device:C
- added C211: 100nF, Capacitor_SMD:C_0805_2012Metric, symbol Device:C
- added FB201: 330R, Inductor_SMD:L_0805_2012Metric, symbol Device:FerriteBead
- added JP201: SolderJumper_2_Open, Jumper:SolderJumper-2_P1.3mm_Open_TrianglePad1.0x1.5mm, symbol Jumper:SolderJumper_2_Open
- added Q201: SSM6K518NU, SSM6K518NU:SOT-1220UDFN6B_TOS, symbol SSM6K518NU:SSM6K518NU
- added U202: LM74700QDDFRQ1, LM74700QDDFRQ1:SOT65P280X110-8N, symbol LM74700QDDFRQ1:LM74700QDDFRQ1
- R204: renamed from R609; value 250R -> 270R
- R205: renamed from R610; value 250R -> 270R
- R206: renamed from R611; value 250R -> 270R
- R208: renamed from R612; value 250R -> 270R
- R209: renamed from R613; value 250R -> 270R
- R210: renamed from R614; value 250R -> 270R
- R211: renamed from R615; value 250R -> 270R
- Y201: renamed from Y601; value 20MHz -> 16MHz
- renumbered C309 to C202, C304 to C205, C601 to C206, C204 to C207, C205 to C208, C602 to C209, C603 to C210, C203 to C212, C201 to C213, C202 to C214, D602 to D201, D201 to D202, D202 to D203, F301 to F201, J301 to J201, J201 to J202, R301 to R201, R302 to R202, R602 to R203, R604 to R207, R201 to R212, R202 to R213, TP306 to TP201, TP305 to TP202, U307 to U201, U306 to U203, U601 to U204, U201 to U205
Connections:
- net +3V3: now also C206.1, C207.1, C208.1, C213.1, C214.1, J202.2, R207.1, U204.18 (AVCC), U204.4 (VCC), U204.6 (VCC), U205.17 (3V3OUT), U205.4 (VCCIO), C211.1
- net +5V: now also C201.1, JP201.2 (B), Q201.1 (D), U202.8 (CATHODE); no longer C206.1, C207.1, C208.1, C213.1, C214.1, J202.2, R207.1, U204.18 (AVCC), U204.4 (VCC), U204.6 (VCC), U205.4 (VCCIO)
- net D+: now also U205.15 (USBD+); no longer U205.16 (USBD-)
- net D-: now also U205.16 (USBD-); no longer U205.15 (USBD+)
- net GND: now also C201.2, C203.2, C211.2, U202.2 (GND)
- net FVBUS: now reaches C205.2, F201.2, U203.5 (VBUS)
- net FVBUS: now also FB201.1
- net CC2: now reaches J201.B5 (CC2), R202.2
- net VBUS: now reaches F201.1, J201.A4 (VBUS), J201.A9 (VBUS), J201.B4 (VBUS), J201.B9 (VBUS)
- net CC1: now reaches J201.A5 (CC1), R201.2
- new net: Q201.2 (G), U202.6 (GATE)
- new net: C204.2, U202.4 (VCAP)
- new net FBFVBUS: C203.1, C204.1, FB201.2, JP201.1 (A), Q201.3 (S), U202.1 (EN), U202.5 (ANODE)
- no-connect marks 27 -> 26
Other:
- note added: "USB-C +3V3"
- note removed: "USB-C +5V +3V3"
- moved on the sheet: C202, C205, F201, J201, R201, R202, TP201, TP202, U201, U203
