File: hardware/keypad/repeater.kicad_sch (KiCad schematic)
At the start: 23 parts, among them U301 SN74HCS4075DR, U302 SN74HCS4075DR, U303 SN74HCS4075DR, U304 NC7SZ00M5X, U305 LMC555CMX/NOPB, U308 NC7SZ00M5X

Commit message: [fix] repeater and sbc shutdown circuit
Fixed repeater and SBC shutdown circuit. Switched +5V VCC to +3.3V. Added C211
Parts:
- removed TP302: White, TestPoint:TestPoint_Keystone_5000-5004_Miniature, symbol Connector:TestPoint
- added C301: 1uF, Capacitor_SMD:C_0805_2012Metric, symbol Device:C
- added Q301: PMV30XPEAR, Package_TO_SOT_SMD:SOT-23-3, symbol PMV30XPEA:PMV30XPEAR
- added U301: 74LVC1G14GW-Q100,1, Package_TO_SOT_SMD:SOT-353_SC-70-5, symbol 74xGxx:74AHC1G14
- C307: renamed from C305; value 1uF -> 10uF
- R301: renamed from R304; now fitted
- renumbered C301 to C302, C310 to C304, C306 to C305, C307 to C306, C302 to C308, C311 to C309, R305 to R302, R306 to R303, R303 to R304, TP303 to TP302, TP304 to TP303, TP307 to TP304, U301 to U302, U308 to U303, U303 to U304, U304 to U305, U305 to U306, U302 to U307
Connections:
- net 3Y_RESET: now also U301.2; no longer U306.4 (R)
- net GATE: now also Q301.1 (G), U301.4; no longer R301.1, TP302.1, U303.1, U305.1, U306.3 (Q)
- net GND: now also C301.2, U301.3 (GND)
- net +5V renamed +3V3
- net +3V3: now also C301.1, Q301.2 (S), U301.5 (VCC); no longer C305.1, C307.1, U306.8 (VCC)
- new net GATED_VCC: C305.1, C307.1, Q301.3 (D), U306.4 (R), U306.8 (VCC)
- new net OSC_GATE: R301.1, TP302.1, U303.1, U305.1, U306.3 (Q)
- no-connect marks 4 -> 2
Other:
- moved on the sheet: C305, C307, R304, TP302, TP303, TP304, U306
