File: hardware/interface-board/production/X2/backups/interface-board/schmitt_triggers.kicad_sch (KiCad schematic)
At the start: 46 parts, among them U901 SN74HC14PWR, U902 SN74HC14PWR, U903 SN74HC14PWR

Commit message: [feat] Revert to Arduino + add PHY
Removed Arduino Due integration. Added W5500 ENET PHY
Parts:
- added D701, D702, D703, D704, D705, D706, D707, D708, D709, D710, D711, D712, D713, D714, D715, D716, D801: BLUE, LED_SMD:LED_1210_3225Metric, symbol Device:LED
- added IC701, IC702, IC703, IC704, IC801: LTV-846S, LTV-846S:LTV846S, symbol LTV-846S:LTV-846S
- added Q701, Q702, Q703, Q704, Q705, Q706, Q707, Q708, Q709, Q710, Q711, Q712, Q713, Q714, Q715, Q716, Q801: BSS138 JI, Package_TO_SOT_SMD:SOT-23, symbol Transistor_FET:BSS138
- added R701, R702, R711, R712, R713, R714, R715, R716, R717, R718, R719, R720, R729, R730, R731, R732, R803: 200R, Resistor_SMD:R_1206_3216Metric, symbol Device:R_US
- added R703, R704, R705, R706, R707, R708, R709, R710, R721, R722, R723, R724, R725, R726, R727, R728, R801: 1K2, Resistor_SMD:R_0805_2012Metric, symbol Device:R_US
- added TP720, TP721, TP722, TP723, TP724, TP725, TP726, TP727, TP728, TP729, TP730, TP731, TP732, TP733, TP734, TP735, TP736, TP737, TP738, TP802: TestPoint, TestPoint:TestPoint_Loop_D2.60mm_Drill1.6mm_Beaded, symbol Connector:TestPoint
Connections:
- net AUTO_BUTTON: now also IC704.6 (K_3); no longer C910.1, R913.2, U903.5 (3A)
- net AUTO_BUTTON*: now also Q715.1 (G), TP732.1
- net ENCODER_BEND_RESET: now also IC701.8 (K_4); no longer C926.1, R918.2, U901.9 (4A)
- net ENCODER_BEND_RESET*: now also Q704.1 (G), TP734.1
- net ENCODER_BEND_SET: now also IC701.6 (K_3); no longer C925.1, R916.2, U901.5 (3A)
- net ENCODER_BEND_SET*: now also Q703.1 (G), TP729.1
- net ENCODER_FEED_RESET: now also IC701.4 (K_2); no longer C924.1, R912.2, U901.3 (2A)
- net ENCODER_FEED_RESET*: now also Q702.1 (G), TP724.1
- net ENCODER_FEED_SET: now also IC701.2 (K_1); no longer C923.1, R907.2, U901.1 (1A)
- net ENCODER_FEED_SET*: now also Q701.1 (G), TP720.1
- net ESTOP: now also IC704.8 (K_4); no longer C905.1, R906.2, U903.11 (5A)
- net ESTOP*: now also U903.8 (4Y), Q716.1 (G), TP737.1; no longer U903.10 (5Y)
- net FUSE: now also IC801.2 (K_1); no longer C912.1, R915.2, U903.9 (4A)
- net FUSE*: now also U903.10 (5Y), Q801.1 (G), TP802.1; no longer U903.8 (4Y)
- net GND: now also IC701.11 (E_3), IC701.13 (E_2), IC701.15 (E_1), IC701.9 (E_4), IC702.11 (E_3), IC702.13 (E_2), IC702.15 (E_1), IC702.9 (E_4), IC703.11 (E_3), IC703.13 (E_2), IC703.15 (E_1), IC703.9 (E_4), IC704.11 (E_3), IC704.13 (E_2), IC704.15 (E_1), IC704.9 (E_4), IC801.15 (E_1), Q701.2 (S), Q702.2 (S), Q703.2 (S), Q704.2 (S), Q705.2 (S), Q706.2 (S), Q707.2 (S), Q708.2 (S), Q709.2 (S), Q710.2 (S), Q711.2 (S), Q712.2 (S), Q713.2 (S), Q714.2 (S), Q715.2 (S), Q716.2 (S), Q801.2 (S), TP728.1, TP733.1, TP738.1
- net PROXIMITY_HEAD_CCW: now also IC704.4 (K_2); no longer C909.1, R911.2, U903.3 (2A)
- net PROXIMITY_HEAD_CCW*: now also Q714.1 (G), TP727.1
- net PROXIMITY_HEAD_CW: now also IC704.2 (K_1); no longer C904.1, R905.2, U903.1 (1A)
- net PROXIMITY_HEAD_CW*: now also Q713.1 (G), TP723.1
- net PROXIMITY_HEAD_IN: now also IC702.4 (K_2); no longer C906.1, R908.2, U901.13 (6A)
- net PROXIMITY_HEAD_IN*: now also Q706.1 (G), TP725.1
- net PROXIMITY_HEAD_LIM: now also IC703.8 (K_4); no longer C908.1, R910.2, U902.13 (6A)
- net PROXIMITY_HEAD_LIM*: now also Q712.1 (G), TP736.1
- net PROXIMITY_HEAD_OUT: now also IC702.2 (K_1); no longer C901.1, R902.2, U901.11 (5A)
- net PROXIMITY_HEAD_OUT*: now also Q705.1 (G), TP721.1
- net PROXIMITY_SHEAR_CUT: now also IC702.8 (K_4); no longer C907.1, R909.2, U902.3 (2A)
- net PROXIMITY_SHEAR_CUT*: now also Q708.1 (G), TP735.1
- net PROXIMITY_SHEAR_HOME: now also IC702.6 (K_3); no longer C902.1, R903.2, U902.1 (1A)
- net PROXIMITY_SHEAR_HOME*: now also Q707.1 (G), TP730.1
- net PROXIMITY_TOOL_IN: now also IC703.2 (K_1); no longer C911.1, R914.2, U902.5 (3A)
- net PROXIMITY_TOOL_IN*: now also Q709.1 (G), TP722.1
- net PROXIMITY_TOOL_OUT: now also IC703.4 (K_2); no longer C913.1, R917.2, U902.9 (4A)
- net PROXIMITY_TOOL_OUT*: now also Q710.1 (G), TP726.1
- net SHEAR_BUTTON: now also IC703.6 (K_3); no longer C903.1, R904.2, U902.11 (5A)
- net SHEAR_BUTTON*: now also Q711.1 (G), TP731.1
- new net: D701.1 (K), Q701.3 (D)
- new net: D705.1 (K), Q705.3 (D)
- new net: D705.2 (A), R713.1
- new net: IC703.3 (A_2), R722.2
- new net: IC703.5 (A_3), R723.2
- new net: IC704.5 (A_3), R727.2
- new net: IC704.3 (A_2), R726.2
- new net: IC701.1 (A_1), R703.2
- new net: IC701.3 (A_2), R704.2
- new net: IC701.5 (A_3), R705.2
- new net: IC701.7 (A_4), R706.2
- new net: D716.2 (A), R732.1
- new net: D702.1 (K), Q702.3 (D)
- new net: IC703.1 (A_1), R721.2
- new net: D712.1 (K), Q712.3 (D)
- new net: D716.1 (K), Q716.3 (D)
- new net: D712.2 (A), R720.1
- new net: D710.1 (K), Q710.3 (D)
- new net: D713.2 (A), R729.1
- new net: D707.2 (A), R715.1
- new net: D711.1 (K), Q711.3 (D)
- new net: IC704.7 (A_4), R728.2
- new net: D713.1 (K), Q713.3 (D)
- new net: IC801.1 (A_1), R801.2
- new net: D706.1 (K), Q706.3 (D)
- new net: D801.2 (A), R803.1
- new net: D711.2 (A), R719.1
- new net: D702.2 (A), R702.1
- new net: IC703.7 (A_4), R724.2
- new net: D704.1 (K), Q704.3 (D)
- new net: D715.2 (A), R731.1
- new net: D706.2 (A), R714.1
- new net: D701.2 (A), R701.1
- new net: D709.2 (A), R717.1
- new net: IC702.1 (A_1), R707.2
- new net: IC702.3 (A_2), R708.2
- new net: IC702.5 (A_3), R709.2
- new net: IC702.7 (A_4), R710.2
- new net: D709.1 (K), Q709.3 (D)
- new net: D801.1 (K), Q801.3 (D)
- new net: IC704.1 (A_1), R725.2
- new net: D704.2 (A), R712.1
- new net: D714.1 (K), Q714.3 (D)
- new net: D703.1 (K), Q703.3 (D)
- new net: D708.2 (A), R716.1
- new net: D707.1 (K), Q707.3 (D)
- new net: D703.2 (A), R711.1
- new net: D710.2 (A), R718.1
- new net: D715.1 (K), Q715.3 (D)
- new net: D714.2 (A), R730.1
- new net: D708.1 (K), Q708.3 (D)
- new net +24V: R703.1, R704.1, R705.1, R706.1, R707.1, R708.1, R709.1, R710.1, R721.1, R722.1, R723.1, R724.1, R725.1, R726.1, R727.1, R728.1, R801.1
- new net +5V: R701.2, R702.2, R711.2, R712.2, R713.2, R714.2, R715.2, R716.2, R717.2, R718.2, R719.2, R720.2, R729.2, R730.2, R731.2, R732.2, R803.2
- new net AUTO_BUTTON**: C910.1, IC704.12 (C_3), R913.2, U903.5 (3A)
- new net ENCODER_BEND_RESET**: C926.1, IC701.10 (C_4), R918.2, U901.9 (4A)
- new net ENCODER_BEND_SET**: C925.1, IC701.12 (C_3), R916.2, U901.5 (3A)
- new net ENCODER_FEED_RESET**: C924.1, IC701.14 (C-2), R912.2, U901.3 (2A)
- new net ENCODER_FEED_SET**: C923.1, IC701.16 (C_1), R907.2, U901.1 (1A)
- new net ESTOP**: C912.1, IC704.10 (C_4), R915.2, U903.9 (4A)
- new net FUSE**: C905.1, IC801.16 (C_1), R906.2, U903.11 (5A)
- new net PROXIMITY_HEAD_CCW**: C909.1, IC704.14 (C-2), R911.2, U903.3 (2A)
- new net PROXIMITY_HEAD_CW**: C904.1, IC704.16 (C_1), R905.2, U903.1 (1A)
- new net PROXIMITY_HEAD_IN**: C906.1, IC702.14 (C-2), R908.2, U901.13 (6A)
- new net PROXIMITY_HEAD_LIM**: C908.1, IC703.10 (C_4), R910.2, U902.13 (6A)
- new net PROXIMITY_HEAD_OUT**: C901.1, IC702.16 (C_1), R902.2, U901.11 (5A)
- new net PROXIMITY_SHEAR_CUT**: C907.1, IC702.10 (C_4), R909.2, U902.3 (2A)
- new net PROXIMITY_SHEAR_HOME**: C902.1, IC702.12 (C_3), R903.2, U902.1 (1A)
- new net PROXIMITY_TOOL_IN**: C911.1, IC703.16 (C_1), R914.2, U902.5 (3A)
- new net PROXIMITY_TOOL_OUT**: C913.1, IC703.14 (C-2), R917.2, U902.9 (4A)
- new net SHEAR_BUTTON**: C903.1, IC703.12 (C_3), R904.2, U902.11 (5A)
- no-connect marks 1 -> 13
Other:
- note added: "1K140: RN73R2ATTD1141D25"
- note added: "Delay"
- note added: "Interrupt LED Indicators"
- note added: "Interrupt LEDS: 2-3V @20mA Half Brightness: 3V @ 10mA = 200R 75% Brightness: 3V @ 15mA = 133.3R"
- note added: "LTV-846S +V Value: 24V LED Voltage Drop: 1.2V LED Current: 20mA Resistor Value: 1K140 Alternative Value: 1K2"
- note added: "Notes"
- note added: "Optoisolators"
- note added: "Test Points"
- moved on the sheet: C901, C902, C903, C904, C905, C906, C907, C908, C909, C910, C911, C912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
